File: Iso.sch (KiCad schematic (older format))
At the start: 15 parts, among them U11 SN74LVC2G14DBV, U12 4N35S, U13 4N35S, U14 SN74LVC2G14DBV

Commit message: First working version
Parts:
- added W3: NET-TIE, conn-test:NET-TIE-0.3mm, symbol NET-TIE
- R43, R44, R45, R46, R47, R48: value 20k -> 22k; BOM RES SMD 20k 1% [0603] -> RES SMD 22k 1% [0603]
Connections:
- net at R41.2, U11.4: now also W3.1; no longer U11.6
- new net: U11.6, W3.2
Other:
- moved on the sheet: C46, C49, R41, R42, R43, R44, R45, R46, R47, R48, R49, U11A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

Commit message: Reannotate component references
Parts:
- renumbered C46 to C54, C49 to C55, R41 to R51, R42 to R52, R43 to R53, R44 to R54, R45 to R55, R46 to R56, R47 to R57, R48 to R58, R49 to R59, U13 to U12, U12 to U13, W3 to W4
Changed lines of the file:
@@
 $EndComp
 $Comp
-L R-0603 R41
+L R-0603 R51
 U 1 1 55D11F5E
 P 3550 4200
-F 0 "R41" V 3362 4200 50  0000 C CNN
+F 0 "R51" V 3362 4200 50  0000 C CNN
 F 1 "100" V 3462 4200 50  0000 C CNN
 F 2 "IPC7351-Nominal:RESC1608X50" H 3550 4200 50  0001 C CNN
@@
 $EndComp
 $Comp
-L R-0603 R49
+L R-0603 R59
 U 1 1 55D12157
 P 7050 4200
-F 0 "R49" V 6862 4200 50  0000 C CNN
+F 0 "R59" V 6862 4200 50  0000 C CNN
 F 1 "100" V 6962 4200 50  0000 C CNN
 F 2 "IPC7351-Nominal:RESC1608X50" H 7050 4200 50  0001 C CNN
@@
 $EndComp
 $Comp
-L 4N35S U13
+L 4N35S U12
 U 1 1 55D121C0
 P 6800 4450
-F 0 "U13" H 6932 4500 50  0000 L CNN
+F 0 "U12" H 6932 4500 50  0000 L CNN
 F 1 "4N35S" H 6932 4400 50  0000 L CNN
 F 2 "smd-semi:SOIC254P1016X460-6" H 6800 4200 60  0001 C CNN
@@
 $EndComp
 $Comp
-L GND #PWR0113
+L GND #PWR117
 U 1 1 55D1227E
 P 6800 4700
-F 0 "#PWR0113" H 6800 4700 30  0001 C CNN
+F 0 "#PWR117" H 6800 4700 30  0001 C CNN
 F 1 "GND" H 6800 4630 30  0001 C CNN
 F 2 "" H 6800 4700 60  0000 C CNN
@@
 $EndComp
 $Comp
-L 4N35S U13
+L 4N35S U12
 U 2 1 55D122B6
 P 5400 4450
-F 0 "U13" H 5533 4500 50  0000 L CNN
+F 0 "U12" H 5533 4500 50  0000 L CNN
 F 1 "4N35S" H 5533 4400 50  0000 L CNN
 F 2 "smd-semi:SOIC254P1016X460-6" H 5400 4200 60  0001 C CNN
@@
 P 5850 4600
 AR Path="/55C7F4BB/55D127F4" Ref="R?"  Part="1"
-AR Path="/55D119A9/55D127F4" Ref="R45"  Part="1"
-F 0 "R45" H 5913 4650 50  0000 L CNN
+AR Path="/55D119A9/55D127F4" Ref="R55"  Part="1"
+F 0 "R55" H 5913 4650 50  0000 L CNN
 F 1 "22k" H 5913 4550 50  0000 L CNN
 F 2 "IPC7351-Nominal:RESC1608X50" H 5850 4600 50  0001 C CNN
@@
 P 5600 4600
 AR Path="/55C7F4BB/55D12849" Ref="R?"  Part="1"
-AR Path="/55D119A9/55D12849" Ref="R44"  Part="1"
-F 0 "R44" H 5663 4650 50  0000 L CNN
+AR Path="/55D119A9/55D12849" Ref="R54"  Part="1"
+F 0 "R54" H 5663 4650 50  0000 L CNN
 F 1 "22k" H 5663 4550 50  0000 L CNN
 F 2 "IPC7351-Nominal:RESC1608X50" H 5600 4600 50  0001 C CNN
@@
 P 5350 4000
 AR Path="/55C7F4BB/55D12985" Ref="R?"  Part="1"
-AR Path="/55D119A9/55D12985" Ref="R43"  Part="1"
-F 0 "R43" H 5413 4050 50  0000 L CNN
+AR Path="/55D119A9/55D12985" Ref="R53"  Part="1"
+F 0 "R53" H 5413 4050 50  0000 L CNN
 F 1 "22k" H 5413 3950 50  0000 L CNN
 F 2 "IPC7351-Nominal:RESC1608X50" H 5350 4000 50  0001 C CNN
@@
 P 5050 2950
 AR Path="/55C7F4BB/55D12B94" Ref="R?"  Part="1"
-AR Path="/55D119A9/55D12B94" Ref="R42"  Part="1"
-F 0 "R42" H 5113 3000 50  0000 L CNN
+AR Path="/55D119A9/55D12B94" Ref="R52"  Part="1"
+F 0 "R52" H 5113 3000 50  0000 L CNN
 F 1 "2k" H 5113 2900 50  0000 L CNN
 F 2 "IPC7351-Nominal:RESC1608X50" H 5050 2950 50  0001 C CNN
@@
 $EndComp
 $Comp
-L 4N35S U12
+L 4N35S U13
 U 1 1 55D132FC
 P 5650 2950
-F 0 "U12" H 5782 3000 50  0000 L CNN
+F 0 "U13" H 5782 3000 50  0000 L CNN
 F 1 "4N35S" H 5782 2900 50  0000 L CNN
 F 2 "smd-semi:SOIC254P1016X460-6" H 5650 2700 60  0001 C CNN
@@
 $EndComp
 $Comp
-L 4N35S U12
+L 4N35S U13
 U 2 1 55D13409
 P 6750 2950
-F 0 "U12" H 6883 3000 50  0000 L CNN
+F 0 "U13" H 6883 3000 50  0000 L CNN
 F 1 "4N35S" H 6883 2900 50  0000 L CNN
 F 2 "smd-semi:SOIC254P1016X460-6" H 6750 2700 60  0001 C CNN
@@
 P 6250 3200
 AR Path="/55C7F4BB/55D13476" Ref="R?"  Part="1"
-AR Path="/55D119A9/55D13476" Ref="R46"  Part="1"
-F 0 "R46" H 6313 3250 50  0000 L CNN
+AR Path="/55D119A9/55D13476" Ref="R56"  Part="1"
+F 0 "R56" H 6313 3250 50  0000 L CNN
 F 1 "22k" H 6313 3150 50  0000 L CNN
 F 2 "IPC7351-Nominal:RESC1608X50" H 6250 3200 50  0001 C CNN
@@
 P 6500 3200
 AR Path="/55C7F4BB/55D134F4" Ref="R?"  Part="1"
-AR Path="/55D119A9/55D134F4" Ref="R47"  Part="1"
-F 0 "R47" H 6563 3250 50  0000 L CNN
+AR Path="/55D119A9/55D134F4" Ref="R57"  Part="1"
+F 0 "R57" H 6563 3250 50  0000 L CNN
 F 1 "22k" H 6563 3150 50  0000 L CNN
 F 2 "IPC7351-Nominal:RESC1608X50" H 6500 3200 50  0001 C CNN
@@
 $EndComp
 $Comp
-L GND #PWR0114
+L GND #PWR113
 U 1 1 55D135D0
 P 6250 3350
-F 0 "#PWR0114" H 6250 3350 30  0001 C CNN
+F 0 "#PWR113" H 6250 3350 30  0001 C CNN
 F 1 "GND" H 6250 3280 30  0001 C CNN
 F 2 "" H 6250 3350 60  0000 C CNN
@@
 $EndComp
 $Comp
-L GND #PWR0115
+L GND #PWR114
 U 1 1 55D13641
 P 6500 3350
-F 0 "#PWR0115" H 6500 3350 30  0001 C CNN
+F 0 "#PWR114" H 6500 3350 30  0001 C CNN
 F 1 "GND" H 6500 3280 30  0001 C CNN
 F 2 "" H 6500 3350 60  0000 C CNN
@@
 $EndComp
 $Comp
-L GND #PWR0116
+L GND #PWR116
 U 1 1 55D1369F
 P 6800 3200
-F 0 "#PWR0116" H 6800 3200 30  0001 C CNN
+F 0 "#PWR116" H 6800 3200 30  0001 C CNN
 F 1 "GND" H 6800 3130 30  0001 C CNN
 F 2 "" H 6800 3200 60  0000 C CNN
@@
 P 6800 2450
 AR Path="/55C7F4BB/55D13723" Ref="R?"  Part="1"
-AR Path="/55D119A9/55D13723" Ref="R48"  Part="1"
-F 0 "R48" H 6863 2500 50  0000 L CNN
+AR Path="/55D119A9/55D13723" Ref="R58"  Part="1"
+F 0 "R58" H 6863 2500 50  0000 L CNN
 F 1 "22k" H 6863 2400 50  0000 L CNN
 F 2 "IPC7351-Nominal:RESC1608X50" H 6800 2450 50  0001 C CNN
@@
 P 2650 3750
 AR Path="/55D163FF" Ref="C?"  Part="1"
-AR Path="/55D119A9/55D163FF" Ref="C46"  Part="1"
-F 0 "C46" H 2763 3800 50  0000 L CNN
+AR Path="/55D119A9/55D163FF" Ref="C54"  Part="1"
+F 0 "C54" H 2763 3800 50  0000 L CNN
 F 1 "1u" H 2763 3700 50  0000 L CNN
 F 2 "IPC7351-Nominal:CAPC2012X70" H 2650 3750 50  0001 C CNN
@@
 $EndComp
 $Comp
-L GND #PWR0117
+L GND #PWR119
 U 1 1 55D177B0
 P 7700 6050
-F 0 "#PWR0117" H 7700 6050 30  0001 C CNN
+F 0 "#PWR119" H 7700 6050 30  0001 C CNN
 F 1 "GND" H 7700 5980 30  0001 C CNN
 F 2 "" H 7700 6050 60  0000 C CNN
@@
 P 8650 5600
 AR Path="/55D17E2D" Ref="C?"  Part="1"
-AR Path="/55D119A9/55D17E2D" Ref="C49"  Part="1"
-F 0 "C49" H 8763 5650 50  0000 L CNN
+AR Path="/55D119A9/55D17E2D" Ref="C55"  Part="1"
+F 0 "C55" H 8763 5650 50  0000 L CNN
 F 1 "1u" H 8763 5550 50  0000 L CNN
 F 2 "IPC7351-Nominal:CAPC2012X70" H 8650 5600 50  0001 C CNN
@@
 $EndComp
 $Comp
-L GND #PWR0118
+L GND #PWR121
 U 1 1 55D17F73
 P 8650 5750
-F 0 "#PWR0118" H 8650 5750 30  0001 C CNN
+F 0 "#PWR121" H 8650 5750 30  0001 C CNN
 F 1 "GND" H 8650 5680 30  0001 C CNN
 F 2 "" H 8650 5750 60  0000 C CNN
@@
 	6800 2300 6800 2350
 $Comp
-L +3.6 #PWR0119
+L +3.6 #PWR120
 U 1 1 55D2B925
 P 8650 5500
-F 0 "#PWR0119" H 8650 5550 30  0001 C CNN
+F 0 "#PWR120" H 8650 5550 30  0001 C CNN
 F 1 "+3.6" H 8650 5613 50  0000 C CNN
 F 2 "" H 8650 5500 60  0000 C CNN
@@
 $EndComp
 $Comp
-L +3.6 #PWR0120
+L +3.6 #PWR118
 U 1 1 55D2B9D4
 P 7700 5200
-F 0 "#PWR0120" H 7700 5250 30  0001 C CNN
+F 0 "#PWR118" H 7700 5250 30  0001 C CNN
 F 1 "+3.6" H 7700 5313 50  0000 C CNN
 F 2 "" H 7700 5200 60  0000 C CNN
@@
 $EndComp
 $Comp
-L +3.6 #PWR0121
+L +3.6 #PWR115
 U 1 1 55D2C1A1
 P 6800 2300
-F 0 "#PWR0121" H 6800 2350 30  0001 C CNN
+F 0 "#PWR115" H 6800 2350 30  0001 C CNN
 F 1 "+3.6" H 6800 2413 50  0000 C CNN
 F 2 "" H 6800 2300 60  0000 C CNN
@@
 $EndComp
 $Comp
-L NET-TIE W3
+L NET-TIE W4
 U 1 1 55D4A1E5
 P 4050 3900
-F 0 "W3" H 4050 4119 50  0000 C CNN
+F 0 "W4" H 4050 4119 50  0000 C CNN
 F 1 "NET-TIE" H 4050 4019 50  0000 C CNN
 F 2 "conn-test:NET-TIE-0.3mm" H 4050 3800 50  0001 C CNN

Commit message: Piles and piles of work
Parts:
- removed C54: 1u, IPC7351-Nominal:CAPC2012X70, symbol C-0805
- removed R52: 2k, IPC7351-Nominal:RESC1608X50, symbol R-0603
- removed R53, R54, R55, R56, R57, R58: 22k, IPC7351-Nominal:RESC1608X50, symbol R-0603
- removed R59: 100, IPC7351-Nominal:RESC1608X50, symbol R-0603
- removed U11, U14: SN74LVC2G14DBV, smd-semi:SOT-23-6, symbol SN74LVC2G14DBV
- removed U12, U13: 4N35S, smd-semi:SOIC254P1016X460-6, symbol 4N35S
- removed W4: NET-TIE, conn-test:NET-TIE-0.3mm, symbol NET-TIE
- added C54, C57: 220p, IPC7351-Nominal:CAPC1608X55, symbol C-0603
- added C56: 1u, IPC7351-Nominal:CAPC2012X70, symbol C-0805
- added R40: 100, IPC7351-Nominal:RESC1608X50, symbol R-0603
- added U12: Si8421, IPC7351-Nominal:SOIC127P600X175-8, symbol Si8421
- R51: BOM RES SMD 100 5% [0603] -> RES SMD 100 1% [0603]
Connections:
- net GND: now also U12.5 (GND2)
- net ISO_GND: now also C54.1, C56.2, C57.1, U12.4 (GND1)
- net ISO_IN: now also R51.2
- net ISO_OUT: now also C57.2, R40.2; no longer R51.1
- net +3.6 renamed +3.3
- net +3.3: now also U12.8 (VCC2)
- new net: C54.2, R51.1, U12.2 (INA)
- new net: R40.1, U12.3 (OUTB)
- new net FROM_ISO_IN: U12.7 (OUTA)
- new net ISO_5V: C56.1, U12.1 (VCC1)
- new net TO_ISO_OUT: U12.6 (INB)
Other:
- note added: "Alternative:\nSi8621"
- moved on the sheet: C55
