File: LocalPwr.sch (KiCad schematic (older format))
At the start: 27 parts, among them U10 TLV702vvDBV, U8 AOZ1282, U9 LM7705

Commit message: First working version
Parts:
- added R59: 2k, IPC7351-Nominal:RESC1608X50, symbol R-0603
- U10: value TLV702vvDBV -> TLV70233DBV; BOM IC TI TLV702vvDBV -> IC TI TLV70233DBV
Connections:
- net GND: now also R59.2
- net +3.3 renamed 3v3
- net 3v3: now also R59.1
- net +3.6 renamed 3v6
- net 3V6_INVERTER renamed 3V6_7705
- net V+ renamed V_IN
- net V- renamed -230mV
Other:
- note added: "Even though @U10 has a very low minimum load\nrequirement, @R59 is necessary as it provides some\nstatic current to permit clamping to the 3.3V rail.\nDo not remove it without ensuring at least 3mA current\nat all times on this rail."
- moved on the sheet: C27, C28, C29, C30, C31, C32, C33, C34, C35, C36, C37, C38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

Commit message: Reannotate component references
Parts:
- renumbered C29 to C40, C40 to C41, C31 to C42, C35 to C43, C36 to C44, C37 to C45, C27 to C46, C38 to C47, C28 to C48, C30 to C49, C39 to C50, C32 to C51, C33 to C52, C34 to C53, E4 to E3, E2 to E4, E3 to E5, R39 to R48, R40 to R49, R59 to R50, TP2 to TP3, TP3 to TP4, TP4 to TP5, U9 to U10, U10 to U9
Other:
- note added: "Even though @U9 has a very low minimum load\nrequirement, @R50 is necessary as it provides some\nstatic current to permit clamping to the 3.3V rail.\nDo not remove it without ensuring at least 3mA current\nat all times on this rail."
- note removed: "Even though @U10 has a very low minimum load\nrequirement, @R59 is necessary as it provides some\nstatic current to permit clamping to the 3.3V rail.\nDo not remove it without ensuring at least 3mA current\nat all times on this rail."

Commit message: Piles and piles of work
Parts:
- removed C40: 33u, IPC7351-Nominal:CAPAE660X570, symbol C-ALUM-660
- removed C48, C51: 22u, IPC7351-Nominal:CAPMP3216X180, symbol C-TANT-3216-18
- removed D5: MBR0520, smd-semi:SOD-123, symbol MBR0520
- added C40: 6u8, IPC7351-Nominal:CAPC3216X70, symbol C-1206
- added C48, C51: 22u, IPC7351-Nominal:CAPC3216X70, symbol C-1206
- added D5: MBR0530, smd-semi:SOD-123, symbol MBR0530
- R48: BOM RES SMD 1k 5% [0603] -> RES SMD 6k98 1% [0603]
Connections:
- net 3V6SW: now also D5.1
- net GND: now also C40.2, C48.2, C51.2, D5.2
- net V_IN: now also C40.1
- net at C52.1, E5.1, U10.6 (VOUT): now also C51.1
- net at U10.7 (CRES): now also C48.1
Other:
- note removed: "-230mV"
Changed lines of the file:
@@
 F 2 "IPC7351-Nominal:RESC1608X50" H 4700 2500 50  0001 C CNN
 F 3 "" H 4700 2550 60  0000 C CNN
-F 4 "Value" H 4700 2500 60  0001 C CNN "Manuf"
-F 5 "RES SMD 1k 5% [0603]" H 5450 3050 60  0001 C CNN "BOM"
+F 4 "RES SMD 6k98 1% [0603]" H 5450 3050 60  0001 C CNN "BOM"
+F 5 "Value" H 4700 2500 60  0001 C CNN "Manuf"
 	1    4700 2500
 	1    0    0    -1
@@
 $EndComp
 $Comp
-L GND #PWR94
+L GND #PWR93
 U 1 1 55CF1E50
 P 4700 3100
-F 0 "#PWR94" H 4700 3100 30  0001 C CNN
+F 0 "#PWR93" H 4700 3100 30  0001 C CNN
 F 1 "GND" H 4700 3030 30  0001 C CNN
 F 2 "" H 4700 3100 60  0000 C CNN
@@
 $EndComp
 $Comp
-L GND #PWR95
+L GND #PWR94
 U 1 1 55CF22FE
 P 5100 2700
-F 0 "#PWR95" H 5100 2700 30  0001 C CNN
+F 0 "#PWR94" H 5100 2700 30  0001 C CNN
 F 1 "GND" H 5100 2630 30  0001 C CNN
 F 2 "" H 5100 2700 60  0000 C CNN
@@
 $EndComp
 $Comp
-L C-ALUM-660 C?
-U 1 1 55CF57EE
-P 2000 2350
-AR Path="/55C7F4BB/55CF57EE" Ref="C?"  Part="1"
-AR Path="/55CEE1A2/55CF57EE" Ref="C40"  Part="1"
-F 0 "C40" H 2113 2400 50  0000 L CNN
-F 1 "33u" H 2113 2300 50  0000 L CNN
-F 2 "IPC7351-Nominal:CAPAE660X570" H 2000 2350 50  0001 C CNN
-F 3 "" H 1990 2325 60  0000 C CNN
-F 4 "DIST DIGIKEY P15444CT-ND" H 2000 2350 60  0001 C CNN "BOM"
-	1    2000 2350
-	1    0    0    -1
-$EndComp
-$Comp
-L GND #PWR92
+L GND #PWR91
 U 1 1 55CF5903
 P 2000 2750
-F 0 "#PWR92" H 2000 2750 30  0001 C CNN
+F 0 "#PWR91" H 2000 2750 30  0001 C CNN
 F 1 "GND" H 2000 2680 30  0001 C CNN
 F 2 "" H 2000 2750 60  0000 C CNN
@@
 	1    0    0    -1
 $EndComp
-Text Notes 3800 2700 0    50   ~ 0
+Text Notes 3750 2700 0    50   ~ 0
 800mV
 $Comp
-L GND #PWR102
+L GND #PWR101
 U 1 1 55CF73E9
 P 7000 5250
-F 0 "#PWR102" H 7000 5250 30  0001 C CNN
+F 0 "#PWR101" H 7000 5250 30  0001 C CNN
 F 1 "GND" H 7000 5180 30  0001 C CNN
 F 2 "" H 7000 5250 60  0000 C CNN
@@
 $EndComp
 $Comp
-L GND #PWR103
+L GND #PWR102
 U 1 1 55CF7440
 P 7000 5650
-F 0 "#PWR103" H 7000 5650 30  0001 C CNN
+F 0 "#PWR102" H 7000 5650 30  0001 C CNN
 F 1 "GND" H 7000 5580 30  0001 C CNN
 F 2 "" H 7000 5650 60  0000 C CNN
@@
 $EndComp
 $Comp
-L GND #PWR107
+L GND #PWR106
 U 1 1 55CF7489
 P 8100 5650
-F 0 "#PWR107" H 8100 5650 30  0001 C CNN
+F 0 "#PWR106" H 8100 5650 30  0001 C CNN
 F 1 "GND" H 8100 5580 30  0001 C CNN
 F 2 "" H 8100 5650 60  0000 C CNN
@@
 	1    8100 5650
 	1    0    0    -1
-$EndComp
-$Comp
-L C-TANT-3216-18 C51
-U 1 1 55CF7735
-P 8200 5300
-F 0 "C51" H 8087 5250 50  0000 R CNN
-F 1 "22u" H 8087 5350 50  0000 R CNN
-F 2 "IPC7351-Nominal:CAPMP3216X180" H 8200 5300 50  0001 C CNN
-F 3 "" H 8190 5275 60  0000 C CNN
-F 4 "DIST DIGIKEY 399-4708-1-ND" H 8200 5300 60  0001 C CNN "BOM"
-	1    8200 5300
-	-1   0    0    1
 $EndComp
 $Comp
@@
 $EndComp
 $Comp
-L GND #PWR109
+L GND #PWR108
 U 1 1 55CF7948
 P 8200 5450
-F 0 "#PWR109" H 8200 5450 30  0001 C CNN
+F 0 "#PWR108" H 8200 5450 30  0001 C CNN
 F 1 "GND" H 8200 5380 30  0001 C CNN
 F 2 "" H 8200 5450 60  0000 C CNN
@@
 $EndComp
 $Comp
-L GND #PWR110
+L GND #PWR109
 U 1 1 55CF79B0
 P 8600 5450
-F 0 "#PWR110" H 8600 5450 30  0001 C CNN
+F 0 "#PWR109" H 8600 5450 30  0001 C CNN
 F 1 "GND" H 8600 5380 30  0001 C CNN
 F 2 "" H 8600 5450 60  0000 C CNN
@@
 	1    0    0    -1
 $EndComp
-Text Notes 8250 5100 0    50   ~ 0
--230mV
-$Comp
-L C-TANT-3216-18 C48
-U 1 1 55CF7E1A
-P 6850 5850
-F 0 "C48" H 6737 5800 50  0000 R CNN
-F 1 "22u" H 6737 5900 50  0000 R CNN
-F 2 "IPC7351-Nominal:CAPMP3216X180" H 6850 5850 50  0001 C CNN
-F 3 "" H 6840 5825 60  0000 C CNN
-F 4 "DIST DIGIKEY 399-4708-1-ND" H 6850 5850 60  0001 C CNN "BOM"
-	1    6850 5850
-	-1   0    0    1
-$EndComp
-$Comp
-L GND #PWR101
+$Comp
+L GND #PWR100
 U 1 1 55CF7ED3
 P 6850 6050
-F 0 "#PWR101" H 6850 6050 30  0001 C CNN
+F 0 "#PWR100" H 6850 6050 30  0001 C CNN
 F 1 "GND" H 6850 5980 30  0001 C CNN
 F 2 "" H 6850 6050 60  0000 C CNN
@@
 $EndComp
 $Comp
-L GND #PWR96
+L GND #PWR95
 U 1 1 55CF8594
 P 5500 2700
-F 0 "#PWR96" H 5500 2700 30  0001 C CNN
+F 0 "#PWR95" H 5500 2700 30  0001 C CNN
 F 1 "GND" H 5500 2630 30  0001 C CNN
 F 2 "" H 5500 2700 60  0000 C CNN
@@
 $EndComp
 $Comp
-L GND #PWR99
+L GND #PWR98
 U 1 1 55CF8971
 P 6600 5450
-F 0 "#PWR99" H 6600 5450 30  0001 C CNN
+F 0 "#PWR98" H 6600 5450 30  0001 C CNN
 F 1 "GND" H 6600 5380 30  0001 C CNN
 F 2 "" H 6600 5450 60  0000 C CNN
@@
 	1    0    0    -1
 $EndComp
-Text Label 6650 5100 0    50   ~ 0
+Text Label 6650 5100 0    40   ~ 0
 3V6_7705
 $Comp
@@
 $EndComp
 $Comp
-L GND #PWR97
+L GND #PWR96
 U 1 1 55CF9273
 P 6100 2700
-F 0 "#PWR97" H 6100 2700 30  0001 C CNN
+F 0 "#PWR96" H 6100 2700 30  0001 C CNN
 F 1 "GND" H 6100 2630 30  0001 C CNN
 F 2 "" H 6100 2700 60  0000 C CNN
@@
 $EndComp
 $Comp
-L GND #PWR112
+L GND #PWR111
 U 1 1 55CF93FF
 P 9100 5450
-F 0 "#PWR112" H 9100 5450 30  0001 C CNN
+F 0 "#PWR111" H 9100 5450 30  0001 C CNN
 F 1 "GND" H 9100 5380 30  0001 C CNN
 F 2 "" H 9100 5450 60  0000 C CNN
@@
 $EndComp
 $Comp
-L GND #PWR100
+L GND #PWR99
 U 1 1 55CFA194
 P 6800 3800
-F 0 "#PWR100" H 6800 3800 30  0001 C CNN
+F 0 "#PWR99" H 6800 3800 30  0001 C CNN
 F 1 "GND" H 6800 3730 30  0001 C CNN
 F 2 "" H 6800 3800 60  0000 C CNN
@@
 $EndComp
 $Comp
-L GND #PWR105
+L GND #PWR104
 U 1 1 55CFA3B7
 P 7600 3500
-F 0 "#PWR105" H 7600 3500 30  0001 C CNN
+F 0 "#PWR104" H 7600 3500 30  0001 C CNN
 F 1 "GND" H 7600 3430 30  0001 C CNN
 F 2 "" H 7600 3500 60  0000 C CNN
@@
 $EndComp
 $Comp
-L GND #PWR106
+L GND #PWR105
 U 1 1 55CFA470
 P 7800 3800
-F 0 "#PWR106" H 7800 3800 30  0001 C CNN
+F 0 "#PWR105" H 7800 3800 30  0001 C CNN
 F 1 "GND" H 7800 3730 30  0001 C CNN
 F 2 "" H 7800 3800 60  0000 C CNN
@@
 $EndComp
 $Comp
-L MBR0520 D5
-U 1 1 55CFAF2C
-P 4150 2500
-F 0 "D5" H 4070 2450 50  0000 R CNN
-F 1 "MBR0520" H 4070 2550 50  0000 R CNN
-F 2 "smd-semi:SOD-123" H 4150 2500 50  0001 C CNN
-F 3 "" H 4150 2500 60  0000 C CNN
-F 4 "Value" H 4150 2500 60  0001 C CNN "Manuf"
-F 5 "SEMI GENERIC MBR0520" H 4900 3050 60  0001 C CNN "BOM"
-	1    4150 2500
-	-1   0    0    1
-$EndComp
-$Comp
-L GND #PWR93
+L GND #PWR92
 U 1 1 55CFB0F5
 P 4150 2650
-F 0 "#PWR93" H 4150 2650 30  0001 C CNN
+F 0 "#PWR92" H 4150 2650 30  0001 C CNN
 F 1 "GND" H 4150 2580 30  0001 C CNN
 F 2 "" H 4150 2650 60  0000 C CNN
@@
 	7250 4700 7400 4700
 $Comp
-L PWR #PWR98
+L PWR #PWR97
 U 1 1 55D4B6EA
 P 6300 2250
-F 0 "#PWR98" H 6300 2250 50  0001 C CNN
+F 0 "#PWR97" H 6300 2250 50  0001 C CNN
 F 1 "PWR" H 6300 2250 50  0001 C CNN
 F 2 "" H 6300 2250 60  0000 C CNN
@@
 Connection ~ 6300 2300
 $Comp
-L PWR #PWR111
+L PWR #PWR110
 U 1 1 55D4C17C
 P 9050 5050
-F 0 "#PWR111" H 9050 5050 50  0001 C CNN
+F 0 "#PWR110" H 9050 5050 50  0001 C CNN
 F 1 "PWR" H 9050 5050 50  0001 C CNN
 F 2 "" H 9050 5050 60  0000 C CNN
@@
 Connection ~ 9050 5100
 $Comp
-L PWR #PWR104
+L PWR #PWR103
 U 1 1 55D3F581
 P 7050 5050
-F 0 "#PWR104" H 7050 5050 50  0001 C CNN
+F 0 "#PWR103" H 7050 5050 50  0001 C CNN
 F 1 "PWR" H 7050 5050 50  0001 C CNN
 F 2 "" H 7050 5050 60  0000 C CNN
@@
 	8200 3300 8200 3500
 $Comp
-L GND #PWR108
+L GND #PWR107
 U 1 1 55D3FE1F
 P 8200 3800
-F 0 "#PWR108" H 8200 3800 30  0001 C CNN
+F 0 "#PWR107" H 8200 3800 30  0001 C CNN
 F 1 "GND" H 8200 3730 30  0001 C CNN
 F 2 "" H 8200 3800 60  0000 C CNN
@@
 	1    0    0    -1
 $EndComp
-Text Notes 6750 4250 0    50   ~ 0
+Text Notes 11100 3700 0    50   ~ 0
 Even though @U9 has a very low minimum load\nrequirement, @R50 is necessary as it provides some\nstatic current to permit clamping to the 3.3V rail.\nDo not remove it without ensuring at least 3mA current\nat all times on this rail.
+$Comp
+L MBR0530 D5
+U 1 1 55DBF46B
+P 4150 2500
+F 0 "D5" H 4070 2450 50  0000 R CNN
+F 1 "MBR0530" H 4070 2550 50  0000 R CNN
+F 2 "smd-semi:SOD-123" H 4150 2500 50  0001 C CNN
+F 3 "" H 4150 2500 60  0000 C CNN
+F 4 "Value" H 4150 2500 60  0001 C CNN "Manuf"
+F 5 "SCHOTTKY MBR0530" H 4900 3050 60  0001 C CNN "BOM"
+	1    4150 2500
+	-1   0    0    1
+$EndComp
+$Comp
+L C-1206 C48
+U 1 1 55DBC55E
+P 6850 5850
+F 0 "C48" H 6963 5900 50  0000 L CNN
+F 1 "22u" H 6963 5800 50  0000 L CNN
+F 2 "IPC7351-Nominal:CAPC3216X70" H 6850 5850 50  0001 C CNN
+F 3 "" H 6840 5825 60  0000 C CNN
+F 4 "CAP MLCC 22u 16V ≥X5R [1206]" H 7650 6400 60  0001 C CNN "BOM"
+F 5 "Value" H 6850 5850 60  0001 C CNN "Manuf"
+	1    6850 5850
+	1    0    0    -1
+$EndComp
+$Comp
+L C-1206 C51
+U 1 1 55DBCC4B
+P 8200 5300
+F 0 "C51" H 8313 5350 50  0000 L CNN
+F 1 "22u" H 8313 5250 50  0000 L CNN
+F 2 "IPC7351-Nominal:CAPC3216X70" H 8200 5300 50  0001 C CNN
+F 3 "" H 8190 5275 60  0000 C CNN
+F 4 "CAP MLCC 22u 16V ≥X5R [1206]" H 9000 5850 60  0001 C CNN "BOM"
+F 5 "Value" H 8200 5300 60  0001 C CNN "Manuf"
+	1    8200 5300
+	1    0    0    -1
+$EndComp
+$Comp
+L C-1206 C40
+U 1 1 55DC13E2
+P 2000 2350
+F 0 "C40" H 2113 2400 50  0000 L CNN
+F 1 "6u8" H 2113 2300 50  0000 L CNN
+F 2 "IPC7351-Nominal:CAPC3216X70" H 2000 2350 50  0001 C CNN
+F 3 "" H 1990 2325 60  0000 C CNN
+F 4 "CAP MLCC 6u8 50V ≥X5R [1206]" H 2800 2900 60  0001 C CNN "BOM"
+F 5 "Value" H 2000 2350 60  0001 C CNN "Manuf"
+	1    2000 2350
+	1    0    0    -1
+$EndComp
 $EndSCHEMATC
