File: LocalPwr.sch (KiCad schematic (older format))
At the start: 28 parts, among them U10 LM7705, U8 AOZ1282, U9 TLV70233DBV

Commit message: Finish PCB
Parts:
- removed C45, C47, C52, C53: 100n, IPC7351-Nominal:CAPC1608X55, symbol C-0603
- removed R48: 6k98, IPC7351-Nominal:RESC1608X50, symbol R-0603
- removed R49, R50: 2k, IPC7351-Nominal:RESC1608X50, symbol R-0603
- added C45, C47, C52, C53: 100n, IPC7351-Nominal:CAPC1005X55, symbol C-0402
- added R48: 6k98, IPC7351-Nominal:RESC1005X40, symbol R-0402
- added R49, R50: 2k, IPC7351-Nominal:RESC1005X40, symbol R-0402
Connections:
- net -230mV: now also C53.1
- net 3V6UF: now also R48.1
- net 3v3: now also R50.1
- net 3v6: now also C45.1, C47.1
- net GND: now also C45.2, C47.2, C52.2, C53.2, R49.2, R50.2
- net at U8.3 (FB): now also R48.2, R49.1
- net at C51.1, E5.1, U10.6 (VOUT): now also C52.1
