File: modpsu.kicad_pcb (KiCad board)
At the start: 2 copper layers, 90 x 90 mm, 420 parts, among them J1 OUT+, J2 OUT-, J3 PDI, J4 IN, J5 IN, J6 OUT, Q1 3904, Q10 AO4805, Q11 4403, Q2 3904, Q3 4403, Q4 4403, Q5 AO4805, Q6 D45H11, Q7 MMBT3904, Q8 PZT3904, Q9 12A, U1 AD8602ARZ, U10 TLV702vvDBV, U11 SN74LVC2G14DBV, U12 4N35S, U13 4N35S, U14 SN74LVC2G14DBV, U2 LM358M, U3 LM393M, U4 SN74LVC2G14DBV, U5 LM393M, U6 ADR380, U7 ATXMEGA32E5-AU, U8 AOZ1282, U9 LM7705

Commit message: First working version
Parts:
- removed MP2: SCREW, mech:SCREW-4-SUPPORTED
- removed R23: 470k, IPC7351-Nominal:RESC1608X50
- removed R52: 20k, IPC7351-Nominal:RESC1608X50
- removed REF**11112, REF**11113, REF**11114, REF**11121, REF**11122, REF**11123, REF**11124, REF**11131, REF**11133, REF**11134, VIA331113 (x3), VIA331121, VIA331122 (x4), VIA331123 (x4), VIA331131, VIA331132 (x4), VIA331133 (x4): VIA-0.8mm, VIA-0.8mm
- removed the REF**12114 at (25.5, 45.0)
- removed the REF**12124 at (26.5, 45.5)
- removed the REF**12144 at (28.5, 45.5)
- removed the VIA331111 at (43.5, 42.5)
- removed the VIA331111 at (54.0, 44.5)
- removed the VIA331111 at (42.0, 44.5)
- removed the VIA331111 at (42.5, 43.5)
- removed the VIA331111 at (45.0, 44.0)
- removed the VIA331111 at (45.0, 45.0)
- removed the VIA331111 at (32.0, 57.0)
- removed the VIA331111 at (41.0, 52.0)
- removed the VIA331111 at (41.5, 51.0)
- removed the VIA331111 at (53.0, 36.5)
- removed the VIA331111 at (52.0, 37.5)
- removed the VIA331111 at (53.5, 39.0)
- removed the VIA331111 at (54.5, 38.5)
- removed the VIA331111 at (54.5, 45.5)
- removed the VIA331111 at (54.0, 46.5)
- removed the VIA331112 at (81.5, 67.5)
- removed the VIA331112 at (62.0, 67.5)
- removed the VIA331112 at (32.0, 59.0)
- removed the VIA33121 at (41.0, 66.0)
- removed the VIA33131 at (42.0, 65.5)
- removed the VIA33132 at (42.0, 66.5)
- added C52: 100n, IPC7351-Nominal:CAPC1608X55, F.Cu at (85.0, 81.0)
- added C53: 100n, IPC7351-Nominal:CAPC1608X55, F.Cu at (85.0, 79.0)
- added C54: 100n, IPC7351-Nominal:CAPC1608X55, F.Cu at (47.0, 15.2)
- added C55: 470u, pth-passive:C-ALUM-10mm, F.Cu at (45.0, 6.50)
- added D3: BAT54AWT, smd-semi:SC-70, F.Cu at (71.0, 6.00)
- added E5: 120, IPC7351-Nominal:INDC1608X95, F.Cu at (60.8, 5.50)
- added J7: BUTTONS, conn-100mil:CONN-100MIL-M-1x3-SHROUD, F.Cu at (83.5, 85.0)
- added Q12: 2N7002PW, smd-semi:SC-70, F.Cu at (66.0, 31.5)
- added R57: 348, IPC7351-Nominal:RESC1608X50, F.Cu at (76.2, 11.0)
- added R58: 22k, IPC7351-Nominal:RESC1608X50, F.Cu at (71.5, 30.0)
- added R59: 2k, IPC7351-Nominal:RESC1608X50, F.Cu at (39.5, 60.5)
- added R60: 1k2, IPC7351-Nominal:RESC6432X70, B.Cu at (63.0, 23.0)
- added R61: 1k2, IPC7351-Nominal:RESC6432X70, B.Cu at (58.0, 23.0)
- added REF**1111111: VIA-0.8mm, VIA-0.8mm, F.Cu at (64.0, 27.5)
- added REF**1111111: VIA-0.8mm, VIA-0.8mm, F.Cu at (63.0, 27.5)
- added REF**1111111: VIA-0.8mm, VIA-0.8mm, F.Cu at (62.0, 27.5)
- added REF**111112: VIA-0.8mm, VIA-0.8mm, F.Cu at (60.5, 53.8)
- added REF**111113: VIA-0.8mm, VIA-0.8mm, F.Cu at (60.5, 54.8)
- added REF**111121: VIA-0.8mm, VIA-0.8mm, F.Cu at (61.5, 53.2)
- added REF**1111211: VIA-0.8mm, VIA-0.8mm, F.Cu at (43.0, 45.0)
- added REF**1111211: VIA-0.8mm, VIA-0.8mm, F.Cu at (31.5, 63.0)
- added REF**1111211: VIA-0.8mm, VIA-0.8mm, F.Cu at (43.5, 66.0)
- added REF**1111211: VIA-0.8mm, VIA-0.8mm, F.Cu at (64.0, 71.5)
- added REF**1111211: VIA-0.8mm, VIA-0.8mm, F.Cu at (42.0, 46.0)
- added REF**1111211: VIA-0.8mm, VIA-0.8mm, F.Cu at (47.5, 45.8)
- added REF**1111211: VIA-0.8mm, VIA-0.8mm, F.Cu at (47.8, 47.8)
- added REF**1111211: VIA-0.8mm, VIA-0.8mm, F.Cu at (46.8, 47.2)
- added REF**1111211: VIA-0.8mm, VIA-0.8mm, F.Cu at (44.5, 49.8)
- added REF**1111211: VIA-0.8mm, VIA-0.8mm, F.Cu at (43.2, 49.8)
- added REF**1111211: VIA-0.8mm, VIA-0.8mm, F.Cu at (44.0, 49.0)
- added REF**1111211: VIA-0.8mm, VIA-0.8mm, F.Cu at (32.5, 51.0)
- added REF**1111212: VIA-0.8mm, VIA-0.8mm, F.Cu at (32.5, 53.0)
- added REF**1111212: VIA-0.8mm, VIA-0.8mm, F.Cu at (31.5, 65.0)
- added REF**1111212: VIA-0.8mm, VIA-0.8mm, F.Cu at (37.0, 64.0)
- added REF**1111212: VIA-0.8mm, VIA-0.8mm, F.Cu at (43.5, 68.0)
- added REF**1111212: VIA-0.8mm, VIA-0.8mm, F.Cu at (64.0, 73.5)
- added REF**1111213: VIA-0.8mm, VIA-0.8mm, F.Cu at (64.0, 75.5)
- added REF**111122: VIA-0.8mm, VIA-0.8mm, F.Cu at (61.5, 54.2)
- added REF**1111221: VIA-0.8mm, VIA-0.8mm, F.Cu at (33.5, 64.0)
- added REF**1111221: VIA-0.8mm, VIA-0.8mm, F.Cu at (39.0, 63.0)
- added REF**1111221: VIA-0.8mm, VIA-0.8mm, F.Cu at (45.5, 67.0)
- added REF**1111221: VIA-0.8mm, VIA-0.8mm, F.Cu at (66.0, 72.5)
- added REF**1111222: VIA-0.8mm, VIA-0.8mm, F.Cu at (33.5, 66.0)
- added REF**1111222: VIA-0.8mm, VIA-0.8mm, F.Cu at (45.5, 69.0)
- added REF**1111222: VIA-0.8mm, VIA-0.8mm, F.Cu at (66.0, 74.5)
- added REF**1111223: VIA-0.8mm, VIA-0.8mm, F.Cu at (66.0, 76.5)
- added REF**111123: VIA-0.8mm, VIA-0.8mm, F.Cu at (55.0, 55.0)
- added REF**111123: VIA-0.8mm, VIA-0.8mm, F.Cu at (70.0, 62.5)
- added REF**111123: VIA-0.8mm, VIA-0.8mm, F.Cu at (61.5, 55.2)
- added REF**111131: VIA-0.8mm, VIA-0.8mm, F.Cu at (64.5, 53.5)
- added REF**111132: VIA-0.8mm, VIA-0.8mm, F.Cu at (62.5, 53.8)
- added REF**111133: VIA-0.8mm, VIA-0.8mm, F.Cu at (62.5, 54.8)
- added REF**111142: VIA-0.8mm, VIA-0.8mm, F.Cu at (63.5, 54.2)
- added REF**111143: VIA-0.8mm, VIA-0.8mm, F.Cu at (63.5, 55.2)
- added REF**12132: VIA-0.8mm, VIA-0.8mm, F.Cu at (31.0, 15.8)
- added REF**12132: VIA-0.8mm, VIA-0.8mm, F.Cu at (31.0, 14.8)
- added REF**12143: VIA-0.8mm, VIA-0.8mm, F.Cu at (31.8, 29.5)
- added REF**12144: VIA-0.8mm, VIA-0.8mm, F.Cu at (31.5, 23.0)
- added REF**12144: VIA-0.8mm, VIA-0.8mm, F.Cu at (30.0, 52.0)
- added REF**12144: VIA-0.8mm, VIA-0.8mm, F.Cu at (30.0, 51.0)
- added REF**12144: VIA-0.8mm, VIA-0.8mm, F.Cu at (30.0, 50.0)
- added TP5: PREREG, conn-test:TEST-SMD-SMALL, F.Cu at (51.5, 4.75)
- added VIA11: VIA-0.8mm, VIA-0.8mm, F.Cu at (75.5, 32.5)
- added VIA12: VIA-0.8mm, VIA-0.8mm, F.Cu at (75.5, 34.5)
- added VIA13: VIA-0.8mm, VIA-0.8mm, F.Cu at (75.5, 36.5)
- added VIA14: VIA-0.8mm, VIA-0.8mm, F.Cu at (75.5, 38.5)
- added VIA21: VIA-0.8mm, VIA-0.8mm, F.Cu at (88.5, 32.5)
- added VIA21: VIA-0.8mm, VIA-0.8mm, F.Cu at (77.5, 32.5)
- added VIA22: VIA-0.8mm, VIA-0.8mm, F.Cu at (88.5, 34.5)
- added VIA22: VIA-0.8mm, VIA-0.8mm, F.Cu at (77.5, 34.5)
- added VIA23: VIA-0.8mm, VIA-0.8mm, F.Cu at (88.5, 36.5)
- added VIA23: VIA-0.8mm, VIA-0.8mm, F.Cu at (77.5, 36.5)
- added VIA24: VIA-0.8mm, VIA-0.8mm, F.Cu at (88.5, 38.5)
- added VIA24: VIA-0.8mm, VIA-0.8mm, F.Cu at (77.5, 38.5)
- added VIA33212: VIA-0.8mm, VIA-0.8mm, F.Cu at (32.5, 61.0)
- added VIA33212: VIA-0.8mm, VIA-0.8mm, F.Cu at (57.2, 4.75)
- added VIA33212: VIA-0.8mm, VIA-0.8mm, F.Cu at (73.0, 84.0)
- added VIA5: VIA-0.8mm, VIA-0.8mm, F.Cu at (64.0, 18.0)
- added VIA5: VIA-0.8mm, VIA-0.8mm, F.Cu at (63.0, 18.0)
- added VIA5: VIA-0.8mm, VIA-0.8mm, F.Cu at (62.0, 18.0)
- C10: value 220p -> 22n
- C11: value 22n -> 220p
- D2: footprint smd-semi:SOT-23 -> smd-semi:SC-70
- DS1, DS2: footprint smd-semi:LED-0603 -> pth-semi:LED-5mm
- DZ1: value 84C24 -> 84B24
- R1, R28: value 2k -> 348
- R12, R15, R17, R18, R34, R38, R43, R44, R45, R46, R47, R48, R50, R53, R8, R9: value 20k -> 22k
- R13, R32, R33, R56: value 330 -> 348
- R24: value 20k -> 2k
- R37: value 470k -> 22k
- U10: value TLV702vvDBV -> TLV70233DBV
- U4: value SN74LVC2G14DBV -> MCP9701-E/TO; footprint smd-semi:SOT-23-6 -> conn-100mil:CONN-100MIL-M-1x3; moved to B.Cu
- W3: footprint conn-test:NET-TIE-1mm -> conn-test:NET-TIE-0.3mm; moved to F.Cu
- moved W3 45.7 mm to (13.8, 81.9), turned to 0 degrees
- moved DS1 26.5 mm to (86.0, 67.0), turned to 90 degrees
- moved DS2 24.7 mm to (86.0, 75.0), turned to 90 degrees
- moved R54 23.4 mm to (83.0, 64.0)
- moved R55 21.9 mm to (83.0, 72.0)
- moved MP1 15.6 mm to (74.0, 72.0)
- moved C16 15.4 mm to (53.0, 40.5), turned to 180 degrees
- moved C51 14.6 mm to (34.0, 41.0), turned to 0 degrees
- moved TP3 14.5 mm to (39.0, 54.0)
- moved U4 11.9 mm to (35.5, 43.8)
- moved C18 11.5 mm to (35.5, 46.0)
- moved R53 10.9 mm to (37.2, 41.0), turned to 0 degrees
- moved VIA33243 10.5 mm to (69.5, 81.5), turned to 180 degrees
- moved J3 10.1 mm to (59.0, 64.0), turned to 180 degrees
- moved U6 10.1 mm to (53.0, 43.5), turned to 0 degrees
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- renumbered REF**11111 to REF**111111
Connections:
- net /LocalPwr/3V6_INVERTER renamed /LocalPwr/3V6_7705
- net Net-(F1-Pad1) renamed /OUT+
- C1 pad 2: PWRGND -> GND
- C14 pad 2: Net-(C14-Pad2) -> /Control/~VLIM
- C15 pad 2: Net-(C15-Pad2) -> /Control/~ILIM
- C19 pad 1: REFGND -> GND
- C2 pad 2: PWRGND -> GND
- C24 pad 2: PWRGND -> GND
- C25 pad 2: PWRGND -> GND
- C26 pad 2: PWRGND -> GND
- C3 pad 1: PWRGND -> GND
- C4 pad 2: PWRGND -> GND
- C41 pad 1: PWRGND -> GND
- C48 pad 2: +3.3 -> /Preregulator/V+F
- C5 pad 1: PWRGND -> GND
- C6 pad 2: PWRGND -> GND
- D1 pad 2: PWRGND -> GND
- J4 pad 2: PWRGND -> GND
- MP1 pad 1: Net-(MP1-Pad1) -> GND
- MP3 pad 1: Net-(MP3-Pad1) -> GND
- MP4 pad 1: Net-(MP4-Pad1) -> GND
- Q4 pad 3: PWRGND -> GND
- Q7 pad 1: Net-(D2-Pad3) -> Net-(D3-Pad2)
- Q8 pad 3: /Linear/P_OUT -> Net-(D3-Pad3)
- R18 pad 2: Net-(D2-Pad3) -> Net-(D3-Pad2)
- R2 pad 2: PWRGND -> GND
- R21 pad 2: PWRGND -> GND
- R22 pad 1: /Linear/P_OUT -> Net-(D3-Pad3)
- R29 pad 1: Net-(C14-Pad2) -> /Control/~VLIM
- R31 pad 1: Net-(C15-Pad2) -> /Control/~ILIM
- R35 pad 1: PWRGND -> GND
- R6 pad 2: /Linear/VSENSE+ -> /Linear/VSENSE-
- R7 pad 2: /Linear/VSENSE- -> /Linear/VSENSE+
- R8 pad 2: /Linear/VSENSE+ -> /Linear/VSENSE-
- R9 pad 2: /Linear/VSENSE- -> /Linear/VSENSE+
- REF**111111 pad 1: PWRGND -> GND
- REF**12111 pad 1: PWRGND -> GND (x2)
- REF**121111 pad 1: PWRGND -> GND
- REF**121112 pad 1: PWRGND -> GND
- REF**121113 pad 1: PWRGND -> GND
- REF**121114 pad 1: PWRGND -> GND
- REF**12112 pad 1: PWRGND -> GND (x2)
- REF**121121 pad 1: PWRGND -> GND
- REF**121122 pad 1: PWRGND -> GND
- REF**121123 pad 1: PWRGND -> GND
- REF**121124 pad 1: PWRGND -> GND
- REF**12113 pad 1: PWRGND -> GND (x5)
- REF**121131 pad 1: PWRGND -> GND
- REF**121132 pad 1: PWRGND -> GND
- REF**121133 pad 1: PWRGND -> GND
- REF**121134 pad 1: PWRGND -> GND
- REF**12114 pad 1: PWRGND -> GND (x5)
- REF**121141 pad 1: PWRGND -> GND
- REF**121142 pad 1: PWRGND -> GND
- REF**121143 pad 1: PWRGND -> GND
- REF**12121 pad 1: PWRGND -> GND (x3)
- REF**12122 pad 1: PWRGND -> GND (x3)
- REF**12123 pad 1: PWRGND -> GND (x6)
- REF**12124 pad 1: PWRGND -> GND (x6)
- REF**12131 pad 1: PWRGND -> GND (x5)
- REF**12132 pad 1: PWRGND -> GND (x4)
- REF**12133 pad 1: PWRGND -> GND (x8)
- REF**12134 pad 1: PWRGND -> GND (x9)
- REF**12141 pad 1: PWRGND -> GND (x4)
- REF**12142 pad 1: PWRGND -> GND (x11)
- REF**12143 pad 1: PWRGND -> GND (x9)
- REF**12144 pad 1: PWRGND -> GND (x7)
- U11 pad 6: Net-(R41-Pad2) -> Net-(U11-Pad6)
- U3 pad 1: Net-(C14-Pad2) -> /Control/~VLIM
- U3 pad 7: Net-(C15-Pad2) -> /Control/~ILIM
- U4 pad 1: Net-(C14-Pad2) -> +3.3
- U4 pad 2: GND -> /Control/TEMP
- U4 pad 3: Net-(C15-Pad2) -> GND
- U7 pad 1: REFGND -> GND
- U7 pad 10: Net-(R55-Pad1) -> GND
- U7 pad 11: GND -> /Control/~EN
- U7 pad 12: GND -> /Control/~VLIM
- U7 pad 13: GND -> /Control/~ILIM
- U7 pad 14: GND -> /Control/~SCR_TRIPPED
- U7 pad 15: GND -> /Control/PREREG_SW
- U7 pad 21: /Control/VLIM -> /Control/TEMP
- U7 pad 22: /Control/ILIM -> +3.3
- U7 pad 23: /Control/~SCR_TRIPPED -> +3.3
- U7 pad 24: /Control/PREREG_SW -> Net-(R50-Pad2)
- U7 pad 27: Net-(R50-Pad2) -> Net-(C52-Pad2)
- U7 pad 28: GND -> Net-(C53-Pad2)
- U7 pad 29: GND -> Net-(R55-Pad1)
- U7 pad 3: Net-(R32-Pad1) -> Net-(R33-Pad1)
- U7 pad 30: GND -> Net-(R54-Pad1)
- U7 pad 4: Net-(R33-Pad1) -> Net-(R32-Pad1)
- U7 pad 5: GND -> REFGND
- U7 pad 9: Net-(R54-Pad1) -> GND
- W3 pad 1: REFGND -> Net-(R41-Pad2)
- W3 pad 2: GND -> Net-(U11-Pad6)
- W4 pad 1: PWRGND -> GND
Routing:
- net PWRGND: track 90.3 -> 0.00 mm, vias 1 -> 0
- net Net-(C52-Pad2): track 0.00 -> 73.7 mm
- net Net-(C53-Pad2): track 0.00 -> 71.7 mm
- net V-: track 62.5 -> 110.3 mm, vias 4 -> 2
- net /Linear/ISENSE: track 89.6 -> 42.2 mm, vias 0 -> 2
- net (no net): track 0.00 -> 40.0 mm
- net +3.3: track 112.7 -> 150.4 mm, vias 8 -> 10
- net /Control/~EN: track 0.00 -> 36.7 mm, vias 0 -> 4
- net REFGND: track 87.8 -> 122.0 mm, vias 7 -> 10
- net Net-(R54-Pad1): track 21.7 -> 50.5 mm
- net Net-(R55-Pad1): track 27.6 -> 55.7 mm
- net /Control/~ILIM: track 0.00 -> 25.1 mm
- net /Control/VSENSE: track 85.1 -> 105.7 mm, vias 7 -> 6
- net /Preregulator/SWNODE: track 19.3 -> 0.00 mm
- net /Linear/P_IN: track 101.2 -> 82.9 mm, vias 2 -> 3
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- added copper zone on B.Cu, net /Linear/P_OUT
- added copper zone on F.Cu, net /Linear/P_OUT
- added copper zone on B.Cu, net /OUT+
- added copper zone on F.Cu, net /OUT+
- removed copper zone on F.Cu, net /LocalPwr/CF+
- removed copper zone on F.Cu, net /LocalPwr/CF-
- removed copper zone on B.Cu, net PWRGND
- removed copper zone on F.Cu, net PWRGND
Other:
- rule pad_to_mask_clearance: 0 -> 0.2
- rule trace_min: 0.2 -> 0.18
- board text added: "+"
- board text added: "-"
- board text added: "20V 3A PSU MODULE"
- board text added: "GND"
- board text added: "MOD12003"
- board text added: "STAR"
- board text added: "TEMPERATURE"
- board text added: "V(T)"
- board text added: "V+"
- board text removed: "BLINKING = FAULT"

Commit message: Reannotate component references
Parts:
- renumbered C22 to C1, C1 to C10, C2 to C11, C3 to C12, C4 to C13, C5 to C14, C6 to C15, C55 to C16, C7 to C17, C8 to C18, C54 to C19, C23 to C2, C42 to C20, C43 to C21, C44 to C22, C45 to C23, C50 to C24, C9 to C25, C47 to C26, C10 to C27, C11 to C28, C14 to C29, C13 to C3, C15 to C30, C18 to C31, C19 to C32, C16 to C33, C17 to C34, C51 to C35, C20 to C36, C52 to C37, C21 to C38, C53 to C39, C12 to C4, C29 to C40, C40 to C41, C31 to C42, C35 to C43, C36 to C44, C37 to C45, C27 to C46, C38 to C47, C28 to C48, C30 to C49, C26 to C5, C39 to C50, C32 to C51, C33 to C52, C34 to C53, C46 to C54, C49 to C55, C24 to C6, C25 to C7, C48 to C8, C41 to C9, D4 to D1, D1 to D2, D2 to D3, D3 to D4, DS2 to DS1, DS1 to DS2, E5 to E1, E1 to E2, E4 to E3, E2 to E4, E3 to E5, J5 to J1, J6 to J2, J4 to J3, J1 to J4, J2 to J5, J3 to J6, L4 to L1, L1 to L2, L2 to L3, L3 to L4, MP3 to MP2, MP4 to MP3, Q10 to Q1, Q6 to Q10, Q7 to Q11, Q8 to Q12, Q9 to Q2, Q1 to Q3, Q2 to Q4, Q3 to Q5, Q4 to Q6, Q5 to Q7, Q11 to Q8, Q12 to Q9, R35 to R1, R3 to R10, R4 to R11, R5 to R12, R6 to R13, R7 to R14, R8 to R15, R9 to R16, R25 to R17, R30 to R18, R10 to R19, R36 to R2, R11 to R20, R12 to R21, R13 to R22, R37 to R23, R38 to R24, R15 to R25, R14 to R26, R16 to R27, R27 to R28, R58 to R29, R2 to R3, R18 to R30, R19 to R31, R57 to R32, R22 to R33, R29 to R34, R31 to R35, R24 to R36, R28 to R37, R26 to R38, R34 to R39, R1 to R4, R56 to R40, R53 to R41, R50 to R42, R51 to R43, R32 to R44, R33 to R45, R55 to R46, R54 to R47, R39 to R48, R40 to R49, R60 to R5, R59 to R50, R41 to R51, R42 to R52, R43 to R53, R44 to R54, R45 to R55, R46 to R56, R47 to R57, R48 to R58, R49 to R59, R61 to R6, R17 to R7, R20 to R8, R21 to R9, TP5 to TP1, TP1 to TP2, TP2 to TP3, TP3 to TP4, TP4 to TP5, U9 to U10, U13 to U12, U12 to U13, U5 to U4, U7 to U5, U4 to U6, U6 to U7, U10 to U9, W4 to W1, W1 to W2, W2 to W3, W3 to W4

Commit message: Piles and piles of work
Parts:
- removed R54, R55, R56, R57, R58: 22k, IPC7351-Nominal:RESC1608X50
- removed R59: 100, IPC7351-Nominal:RESC1608X50
- removed the REF**1111211 at (31.5, 63.0)
- removed the REF**1111211 at (64.0, 71.5)
- removed the REF**1111211 at (47.5, 45.8)
- removed the REF**1111211 at (47.8, 47.8)
- removed the REF**1111211 at (46.8, 47.2)
- removed the REF**1111211 at (44.5, 49.8)
- removed the REF**1111211 at (44.0, 49.0)
- removed the REF**1111212 at (43.5, 68.0)
- removed the REF**1111212 at (64.0, 73.5)
- removed REF**1111213, REF**1111223: VIA-0.8mm, VIA-0.8mm
- removed the REF**1111221 at (66.0, 72.5)
- removed the REF**1111222 at (66.0, 74.5)
- removed the REF**12113 at (25.5, 44.0)
- removed the REF**12123 at (26.5, 44.5)
- removed the REF**12133 at (27.5, 44.0)
- removed the REF**12142 at (32.0, 9.50)
- removed U11, U14: SN74LVC2G14DBV, smd-semi:SOT-23-6
- removed U13: 4N35S, smd-semi:SOIC254P1016X460-6
- removed the VIA33212 at (32.5, 61.0)
- removed W4: NET-TIE, conn-test:NET-TIE-0.3mm
- added C56: 1u, IPC7351-Nominal:CAPC2012X70, F.Cu at (19.0, 79.0)
- added C57: 220p, IPC7351-Nominal:CAPC1608X55, F.Cu at (8.00, 83.0)
- added C58: 1k/1kV, IPC7351-Nominal:CAPC3216X70, F.Cu at (65.5, 71.5)
- added J8: DEVEL, conn-100mil:CONN-100MIL-M-1x3, F.Cu at (35.0, 73.2)
- added JP3: JUMPER, conn-100mil:CONN-100MIL-M-1x2, F.Cu at (35.8, 82.0)
- added REF**1111111: VIA-0.8mm, VIA-0.8mm, F.Cu at (59.0, 27.5)
- added REF**1111111: VIA-0.8mm, VIA-0.8mm, F.Cu at (58.0, 27.5)
- added REF**1111211: VIA-0.8mm, VIA-0.8mm, F.Cu at (40.0, 56.5)
- added REF**1111211: VIA-0.8mm, VIA-0.8mm, F.Cu at (38.5, 56.5)
- added REF**1111211: VIA-0.8mm, VIA-0.8mm, F.Cu at (38.5, 55.0)
- added REF**111142: VIA-0.8mm, VIA-0.8mm, F.Cu at (66.5, 52.0)
- added SYM1: OSHW-SCHEM-PCB6mm, mech:OSHW-6mm, F.Cu at (4.00, 86.0)
- added TP10: ISET, conn-test:TEST-SMD-SMALL, F.Cu at (59.8, 37.5)
- added TP11: VDRIVE, conn-test:TEST-SMD-SMALL, F.Cu at (68.5, 31.8)
- added TP12: IDRIVE, conn-test:TEST-SMD-SMALL, F.Cu at (60.2, 33.1)
- added TP13: DRIVE, conn-test:TEST-SMD-SMALL, F.Cu at (64.5, 30.0)
- added TP14: SW, conn-test:TEST-SMD-SMALL, F.Cu at (39.2, 30.5)
- added TP6: OVP_TH, conn-test:TEST-SMD-SMALL, F.Cu at (42.8, 17.2)
- added TP7: VSENSE, conn-test:TEST-SMD-SMALL, F.Cu at (56.2, 53.5)
- added TP8: VSET, conn-test:TEST-SMD-SMALL, F.Cu at (69.0, 39.5)
- added TP9: ISENSE, conn-test:TEST-SMD-SMALL, F.Cu at (56.0, 49.2)
- added VIA3112: VIA-0.8mm, VIA-0.8mm, F.Cu at (20.5, 86.0)
- added VIA3112: VIA-0.8mm, VIA-0.8mm, F.Cu at (17.5, 80.5)
- added VIA3112: VIA-0.8mm, VIA-0.8mm, F.Cu at (32.2, 84.5)
- added VIA3112: VIA-0.8mm, VIA-0.8mm, F.Cu at (32.2, 85.5)
- added VIA3112: VIA-0.8mm, VIA-0.8mm, F.Cu at (31.5, 85.0)
- added VIA3112: VIA-0.8mm, VIA-0.8mm, F.Cu at (32.0, 78.5)
- added VIA3112: VIA-0.8mm, VIA-0.8mm, F.Cu at (33.0, 80.0)
- added VIA3112: VIA-0.8mm, VIA-0.8mm, F.Cu at (20.5, 85.0)
- added VIA3112: VIA-0.8mm, VIA-0.8mm, F.Cu at (19.5, 85.5)
- added VIA3112: VIA-0.8mm, VIA-0.8mm, F.Cu at (19.5, 86.5)
- added VIA3112: VIA-0.8mm, VIA-0.8mm, F.Cu at (16.0, 73.5)
- added VIA3112: VIA-0.8mm, VIA-0.8mm, F.Cu at (16.0, 75.5)
- added VIA3112: VIA-0.8mm, VIA-0.8mm, F.Cu at (18.5, 80.5)
- added VIA3112: VIA-0.8mm, VIA-0.8mm, F.Cu at (18.5, 81.5)
- added VIA3112: VIA-0.8mm, VIA-0.8mm, F.Cu at (17.5, 81.5)
- added VIA331311: VIA-0.8mm, VIA-0.8mm, F.Cu at (61.0, 70.5)
- added VIA331312: VIA-0.8mm, VIA-0.8mm, F.Cu at (61.0, 71.5)
- added VIA331313: VIA-0.8mm, VIA-0.8mm, F.Cu at (61.0, 72.5)
- added VIA331321: VIA-0.8mm, VIA-0.8mm, F.Cu at (62.0, 71.0)
- added VIA331322: VIA-0.8mm, VIA-0.8mm, F.Cu at (62.0, 72.0)
- added VIA331323: VIA-0.8mm, VIA-0.8mm, F.Cu at (62.0, 73.0)
- added VIA331331: VIA-0.8mm, VIA-0.8mm, F.Cu at (61.0, 73.5)
- added VIA331332: VIA-0.8mm, VIA-0.8mm, F.Cu at (61.0, 74.5)
- added VIA331333: VIA-0.8mm, VIA-0.8mm, F.Cu at (61.0, 75.5)
- added VIA33212: VIA-0.8mm, VIA-0.8mm, F.Cu at (67.0, 57.5)
- added VIA33212: VIA-0.8mm, VIA-0.8mm, F.Cu at (43.5, 68.0)
- added VIA5: VIA-0.8mm, VIA-0.8mm, F.Cu at (57.0, 18.0)
- added VIA5: VIA-0.8mm, VIA-0.8mm, F.Cu at (59.0, 18.0)
- added VIA5: VIA-0.8mm, VIA-0.8mm, F.Cu at (58.0, 18.0)
- C10: value 100p -> 220p
- C40, C7: value 33u -> 6u8; footprint IPC7351-Nominal:CAPAE660X570 -> IPC7351-Nominal:CAPC3216X70
- C48, C51: footprint IPC7351-Nominal:CAPMP3216X180 -> IPC7351-Nominal:CAPC3216X70
- C54: value 1u -> 220p; footprint IPC7351-Nominal:CAPC2012X70 -> IPC7351-Nominal:CAPC1608X55
- C6: value 33u -> 470u; footprint IPC7351-Nominal:CAPAE660X570 -> pth-passive:C-ALUM-10mm
- D5: value MBR0520 -> MBR0530
- J1, J2: footprint conn-100mil:CONN-100MIL-M-1x3-SHROUD -> conn-100mil:CONN-100MIL-M-1x4-SHROUD
- R28, R5, R6: value 1k2 -> 1k
- R40: value 348 -> 100
- R52: value 2k -> 470k
- R53: value 22k -> 470k
- U1: value AD8602ARZ -> OPA2376AID
- U12: value 4N35S -> Si8421; footprint smd-semi:SOIC254P1016X460-6 -> IPC7351-Nominal:SOIC127P600X175-8
- U5: value ATXMEGA32E5-AU -> ATXMEGA8E5-AU
- moved R52 49.3 mm to (66.5, 74.5), turned to 0 degrees
- moved R53 48.0 mm to (63.0, 74.5)
- moved R40 42.0 mm to (11.2, 83.0), turned to 180 degrees
- moved R51 12.8 mm to (18.0, 72.8), turned to 180 degrees
- moved VIA33232 8.86 mm to (62.0, 85.5)
- moved C7 8.75 mm to (24.4, 33.8)
- moved VIA33222 8.62 mm to (63.2, 85.0)
- moved VIA33223 8.62 mm to (63.2, 84.0)
- moved R50 8.06 mm to (35.5, 53.5), turned to 0 degrees
- moved VIA33212 7.78 mm to (67.5, 78.5)
- moved C6 7.50 mm to (24.5, 42.5)
- moved VIA33241 6.80 mm to (75.5, 85.0)
- moved C53 6.37 mm to (74.8, 82.8), turned to 270 degrees
- moved C48 6.10 mm to (67.5, 83.5), turned to 270 degrees
- moved VIA33243 6.01 mm to (69.8, 87.5)
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Connections:
- C48 pad 1: GND -> Net-(C48-Pad1)
- C48 pad 2: Net-(C48-Pad2) -> GND
- C51 pad 1: GND -> Net-(C51-Pad1)
- C51 pad 2: Net-(C51-Pad2) -> GND
- C52 pad 1: Net-(C51-Pad2) -> Net-(C51-Pad1)
- C54 pad 1: /Iso/ISO_3V3 -> /Iso/ISO_GND
- C54 pad 2: /Iso/ISO_GND -> Net-(C54-Pad2)
- C55 pad 1: +3.6 -> +3.3
- E5 pad 1: Net-(C51-Pad2) -> Net-(C51-Pad1)
- J1 pad 1: /Iso/ISO_3V3 -> /Iso/ISO_GND
- J2 pad 1: /Iso/ISO_3V3 -> /Iso/ISO_GND
- MP1 pad 1: GND -> /PAD_MP1
- MP2 pad 1: GND -> /PAD_MP2
- MP3 pad 1: GND -> /PAD_MP3
- R40 pad 2: /Iso/OUT -> /Iso/ISO_OUT
- R51 pad 1: /Iso/ISO_OUT -> Net-(C54-Pad2)
- R51 pad 2: Net-(R51-Pad2) -> /Iso/ISO_IN
- R52 pad 1: /Iso/ISO_3V3 -> Net-(R52-Pad1)
- R52 pad 2: /Iso/ISO_IN -> /PAD_MP1
- R53 pad 1: /Iso/ISO_3V3 -> GND
- R53 pad 2: Net-(R53-Pad2) -> Net-(R52-Pad1)
- U10 pad 6: Net-(C51-Pad2) -> Net-(C51-Pad1)
- U10 pad 7: Net-(C48-Pad2) -> Net-(C48-Pad1)
- U12 pad 1: Net-(R59-Pad1) -> /Iso/ISO_5V
- U12 pad 2: GND -> Net-(C54-Pad2)
- U12 pad 3: (no net) -> Net-(R40-Pad1)
- U12 pad 5: Net-(R53-Pad2) -> GND
- U12 pad 6: Net-(R54-Pad1) -> /Iso/TO_ISO_OUT
- U5 pad 25: /Iso/IN -> /Iso/TO_ISO_OUT
- U5 pad 26: Net-(R40-Pad1) -> /Control/RX
Routing:
- net /Iso/ISO_3V3: track 46.5 -> 0.00 mm
- net /Iso/TO_ISO_OUT: track 0.00 -> 43.5 mm, vias 0 -> 2
- net /Iso/ISO_5V: track 0.00 -> 38.9 mm
- net /Control/RX: track 0.00 -> 33.4 mm
- net +3.3: track 150.4 -> 182.4 mm
- net /Iso/OUT: track 29.9 -> 0.00 mm, vias 2 -> 0
- net /Iso/IN: track 28.0 -> 0.00 mm
- net Net-(C54-Pad2): track 0.00 -> 16.3 mm
- net /PAD_MP1: track 0.00 -> 14.0 mm
- net +3.6: track 74.6 -> 62.1 mm
- net GND: track 72.5 -> 60.5 mm, vias 22 -> 19
- net Net-(C51-Pad1): track 0.00 -> 11.1 mm
- net Net-(R53-Pad2): track 9.72 -> 0.00 mm
- net /Iso/FROM_ISO_IN: track 0.00 -> 8.63 mm
- net REFGND: track 122.0 -> 130.6 mm
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Other:
- outline, holes or cut-outs redrawn
- net class Default: clearance 0.18 -> 0.2
- rule trace_clearance: 0.18 -> 0.2
- board text added: "--"
- board text added: "CLK"
- board text added: "CPOHL1.0 NIHLABS MOD12003 REV A: 201508 ASSY REV:"
- board text added: "DAT"
- board text added: "INSUL SCREW ONLY!"
- board text added: "REF"
- board text added: "~RST"
