File: Control.sch (KiCad schematic (older format))
At the start: 26 parts, among them J6 PDI, J7 BUTTONS, U5 ATXMEGA8E5-AU, U6 MCP9701-E/TO, U7 ADR380

Commit message: Finish PCB
Parts:
- removed C31, C32, C33, C34, C35, C36, C37, C38, C39: 100n, IPC7351-Nominal:CAPC1608X55, symbol C-0603
- removed R39, R41, R42: 22k, IPC7351-Nominal:RESC1608X50, symbol R-0603
- removed R43, R46, R47: 2k, IPC7351-Nominal:RESC1608X50, symbol R-0603
- removed R44, R45: 348, IPC7351-Nominal:RESC1608X50, symbol R-0603
- removed U5: ATXMEGA8E5-AU, IPC7351-Nominal:QFP80P900X900X120-32, symbol ATXMEGA8E5-AU
- added C31, C32, C33, C34, C35, C36, C37, C38, C39, C59: 100n, IPC7351-Nominal:CAPC1005X55, symbol C-0402
- added E6: 120, IPC7351-Nominal:INDC1608X95, symbol BEAD-0603
- added R39, R42: 22k, IPC7351-Nominal:RESC1005X40, symbol R-0402
- added R41: 470k, IPC7351-Nominal:RESC1005X40, symbol R-0402
- added R43, R46, R47: 2k, IPC7351-Nominal:RESC1005X40, symbol R-0402
- added R44, R45: 348, IPC7351-Nominal:RESC1005X40, symbol R-0402
- added U11: MAX5215, IPC7351-Nominal:SOP65P490X110-8, symbol MAX5215
- added U5: ATXMEGA32E5-M4U, smd-semi:QFN40P400X400X55-33, symbol ATXMEGA32E5-M4U
Connections:
- net +3.3: now also C31.1, E6.1, R39.2, U5.17 (V+)
- net +3.3A: now also C32.1, C59.1, U11.5 (~AUX), U11.7 (V+), U5.32 (V+A); no longer U7.1 (IN)
- net GND: now also C31.2, C32.2, C35.2, C37.2, C39.2, R43.2, U5.1 (GNDA), U5.18 (GND), U5.33 (GND(EP)), U5.9 (OC4D/TX0/MOSI/PC7)
- net ISENSE: now also U5.3 (ADC3/DAC1/PA3)
- net ISET: now also C38.1, R44.1
- net OVPTH_PWM: now also R41.2, U5.15 (OC4B/SCL/PC1)
- net OVP_THRESH: now also C35.1, R41.1
- net PDI_C: now also R39.1, U5.8 (PDI_C/~RST)
- net PDI_D: now also U5.7 (PDI_D)
- net PREREG_SW: now also U5.14 (OC4C/RX0/PC2)
- net REFGND: now also C33.2, C34.2, C36.2, C38.2, C59.2, U11.2 (ADDR), U11.8 (GND), U5.5 (ADC1/PA1)
- net RX: now also U5.22 (ADC14/RX0/PD6)
- net TEMP: now also U5.29 (ADC7/PA7)
- net TX: now also U5.21 (ADC15/TX0/PD7)
- net VPREREG: now also R42.1
- net VREF: now also C34.1, U11.1 (REF), U5.6 (ADC0/AREF/PA0)
- net VSENSE: now also U5.2 (ADC4/PA4)
- net VSET: now also C36.1, R45.1
- net ~EN: now also U5.10 (OC4C/RX0/MISO/PC6)
- net ~ILIM: now also U5.12 (OC4A/OC5A/~SS~/PC4)
- net ~SCR_TRIPPED: now also U5.13 (OC4D/TX0/PC3)
- net ~VLIM: now also U5.11 (OC4B/OC5B/SCK/PC5)
- net at DS2.2: now also R47.2
- net at DS1.2: now also R46.2
- net BTN1: now reaches J7.2
- net BTN1: now also C39.1, U5.20 (PR0/XTAL2)
- net BTN2: now reaches J7.3
- net BTN2: now also C37.1, U5.23 (ADC13/OC5B/PD5)
- new net: C33.1, E6.2, U7.1 (IN)
- new net: R42.2, R43.1, U5.24 (ADC12/OC5A/PD4)
- new net: R44.2, U5.4 (ADC2/DAC0/PA2)
- new net: R45.2, U11.6 (OUT)
- new net LEDCC: R46.1, U5.25 (ADC11/TX0/PD3)
- new net LEDCV: R47.1, U5.26 (ADC10/RX0/PD2)
- new net SCL: U11.3 (SCL), U5.27 (ADC9/SCL/PD1)
- new net SDA: U11.4 (SDA), U5.28 (ADC8/SDA/PD0)
Other:
- moved on the sheet: DS1, DS2, J7, U6

Commit message: Add LEDs and mode reporting
Parts:
- renumbered DS2 to DS1, DS1 to DS2
Connections:
- net at DS1.2: now also R46.2; no longer R47.2
- net at DS2.2: now also R47.2; no longer R46.2
Other:
- moved on the sheet: DS1, DS2
Changed lines of the file:
@@
+$EndComp
+$Comp
+L LED-5MM DS1
+U 1 1 55D2BF55
+P 8700 5750
+F 0 "DS1" H 8850 5800 50  0000 L CNN
+F 1 "CV" H 8850 5700 50  0000 L CNN
+F 2 "pth-semi:LED-5mm" H 8700 5750 50  0001 C CNN
+F 3 "" H 8700 5750 60  0000 C CNN
+F 4 "LED GREEN [5mm]" H 9550 6300 60  0001 C CNN "BOM"
+	1    8700 5750
+	1    0    0    -1
 $EndComp
 $Comp
 L LED-5MM DS2
-U 1 1 55D2BF55
+U 1 1 55D2C1B3
 P 9100 5750
 F 0 "DS2" H 9250 5800 50  0000 L CNN
-F 1 "CV" H 9250 5700 50  0000 L CNN
+F 1 "CC" H 9250 5700 50  0000 L CNN
 F 2 "pth-semi:LED-5mm" H 9100 5750 50  0001 C CNN
 F 3 "" H 9100 5750 60  0000 C CNN
-F 4 "LED GREEN [5mm]" H 9950 6300 60  0001 C CNN "BOM"
+F 4 "LED RED [5mm]" H 9950 6300 60  0001 C CNN "BOM"
 	1    9100 5750
 	1    0    0    -1
 $EndComp
-$Comp
-L LED-5MM DS1
-U 1 1 55D2C1B3
-P 8700 5750
-F 0 "DS1" H 8850 5800 50  0000 L CNN
-F 1 "CC" H 8850 5700 50  0000 L CNN
-F 2 "pth-semi:LED-5mm" H 8700 5750 50  0001 C CNN
-F 3 "" H 8700 5750 60  0000 C CNN
-F 4 "LED RED [5mm]" H 9550 6300 60  0001 C CNN "BOM"
-	1    8700 5750
-	1    0    0    -1
-$EndComp

Commit message: Fix output blip
Add a bodge wire to prototype to allow the MCU to force the regulator
into saturation-low
Connections:
- net FORCE_SAT_L: now reaches U5.31 (ADC5/PA5)
Changed lines of the file:
@@
 Wire Wire Line
 	7000 3400 7000 1100
+Text HLabel 6300 3200 2    50   Output ~ 0
+FORCE_SAT_L
+Wire Wire Line
+	6300 3200 5400 3200
 $EndSCHEMATC
