File: Preregulator.sch (KiCad schematic (older format))
At the start: 30 parts, among them Q3 3904, Q4 3904, Q5 4403, Q6 4403, Q7 AO4805

Commit message: Documentation editing
Other:
- moved on the sheet: C8
Changed lines of the file:
@@
 U 1 1 55C7F6FF
 P 4050 3300
-F 0 "Q5" H 4150 3250 50  0000 L CNN
-F 1 "4403" H 4150 3150 50  0000 L CNN
+F 0 "Q5" H 4141 3350 50  0000 L CNN
+F 1 "4403" H 4141 3250 50  0000 L CNN
 F 2 "smd-semi:SOT-23" H 4050 3450 50  0001 C CNN
 F 3 "" H 4050 3300 60  0000 C CNN
@@
 P_OUT
 Wire Wire Line
-	5300 4100 6350 4100
+	5300 4100 6100 4100
+Wire Wire Line
+	6100 4100 6350 4100
 Wire Wire Line
 	6900 4100 6900 4200
@@
 Connection ~ 6900 4100
 Wire Wire Line
-	5300 3850 5300 4500
+	5300 3850 5300 3900
+Wire Wire Line
+	5300 3900 5300 4100
+Wire Wire Line
+	5300 4100 5300 4500
 Connection ~ 5300 4100
 Wire Wire Line
@@
 	6100 4800 6100 4700
 Wire Wire Line
-	6550 4100 7000 4100
+	6550 4100 6900 4100
+Wire Wire Line
+	6900 4100 7000 4100
 Wire Wire Line
 	7300 4200 7300 4100
 Wire Wire Line
-	7200 4100 7900 4100
+	7200 4100 7300 4100
+Wire Wire Line
+	7300 4100 7700 4100
+Wire Wire Line
+	7700 4100 7800 4100
+Wire Wire Line
+	7800 4100 7900 4100
 Wire Wire Line
 	7300 4500 7300 4400
@@
 	6700 4650 6700 4450
 Wire Wire Line
-	4100 3400 4100 4000
-Wire Wire Line
-	4100 3700 5150 3700
+	4100 3400 4100 3700
+Wire Wire Line
+	4100 3700 4100 3800
+Wire Wire Line
+	4100 3800 4100 4000
+Wire Wire Line
+	4100 3700 5100 3700
+Wire Wire Line
+	5100 3700 5150 3700
 Connection ~ 4100 3700
 Wire Wire Line
-	3800 3200 3800 3450
+	3800 3200 3800 3300
+Wire Wire Line
+	3800 3300 3800 3450
 Wire Wire Line
 	3800 3300 3950 3300
@@
 	3800 2900 3800 3000
 Wire Wire Line
-	2100 2900 5450 2900
-Wire Wire Line
-	5300 2900 5300 3650
+	2100 2900 2300 2900
+Wire Wire Line
+	2300 2900 2700 2900
+Wire Wire Line
+	2700 2900 3400 2900
+Wire Wire Line
+	3400 2900 3800 2900
+Wire Wire Line
+	3800 2900 4100 2900
+Wire Wire Line
+	4100 2900 4450 2900
+Wire Wire Line
+	4450 2900 5300 2900
+Wire Wire Line
+	5300 2900 5450 2900
+Wire Wire Line
+	5300 2900 5300 3550
+Wire Wire Line
+	5300 3550 5300 3650
 Wire Wire Line
 	4100 3200 4100 2900
@@
 	3650 3550 3400 3550
 Wire Wire Line
-	3400 3300 3400 4400
+	3400 3300 3400 3550
+Wire Wire Line
+	3400 3550 3400 4100
+Wire Wire Line
+	3400 4100 3400 4400
 Wire Wire Line
 	3400 4100 3950 4100
@@
 	3400 4700 3400 4600
 Wire Wire Line
-	4100 4200 4100 5350
+	4100 4200 4100 5250
+Wire Wire Line
+	4100 5250 4100 5350
 Wire Wire Line
 	4100 5250 3400 5250
 Connection ~ 4100 5250
 Wire Wire Line
-	1400 4500 3250 4500
-Wire Wire Line
-	8100 4100 9600 4100
+	1400 4500 2700 4500
+Wire Wire Line
+	2700 4500 3250 4500
+Wire Wire Line
+	8100 4100 8200 4100
+Wire Wire Line
+	8200 4100 8300 4100
+Wire Wire Line
+	8300 4100 8700 4100
+Wire Wire Line
+	8700 4100 8800 4100
+Wire Wire Line
+	8800 4100 8900 4100
+Wire Wire Line
+	8900 4100 9100 4100
+Wire Wire Line
+	9100 4100 9600 4100
 Wire Wire Line
 	3400 4950 3400 4900
@@
 $EndComp
 Wire Wire Line
-	1400 2900 1900 2900
+	1400 2900 1600 2900
+Wire Wire Line
+	1600 2900 1900 2900
 $Comp
 L C-ALUM-10mm C5
@@
 	5600 3900 5600 3850
 Wire Wire Line
-	5300 3900 5600 3900
+	5300 3900 5350 3900
+Wire Wire Line
+	5350 3900 5550 3900
+Wire Wire Line
+	5550 3900 5600 3900
 Connection ~ 5300 3900
 Wire Wire Line
@@
 	5450 3250 5450 3200
 $Comp
-L GND #PWR21
+L GND #PWR016
 U 1 1 55D3B7DF
 P 5300 4800
-F 0 "#PWR21" H 5300 4800 30  0001 C CNN
+F 0 "#PWR016" H 5300 4800 30  0001 C CNN
 F 1 "GND" H 5300 4730 30  0001 C CNN
 F 2 "" H 5300 4800 60  0000 C CNN
@@
 $EndComp
 $Comp
-L GND #PWR23
+L GND #PWR017
 U 1 1 55D3B842
 P 6100 4800
-F 0 "#PWR23" H 6100 4800 30  0001 C CNN
+F 0 "#PWR017" H 6100 4800 30  0001 C CNN
 F 1 "GND" H 6100 4730 30  0001 C CNN
 F 2 "" H 6100 4800 60  0000 C CNN
@@
 $EndComp
 $Comp
-L GND #PWR24
+L GND #PWR018
 U 1 1 55D3B89E
 P 6900 4500
-F 0 "#PWR24" H 6900 4500 30  0001 C CNN
+F 0 "#PWR018" H 6900 4500 30  0001 C CNN
 F 1 "GND" H 6900 4430 30  0001 C CNN
 F 2 "" H 6900 4500 60  0000 C CNN
@@
 $EndComp
 $Comp
-L GND #PWR25
+L GND #PWR019
 U 1 1 55D3B8FA
 P 7300 4500
-F 0 "#PWR25" H 7300 4500 30  0001 C CNN
+F 0 "#PWR019" H 7300 4500 30  0001 C CNN
 F 1 "GND" H 7300 4430 30  0001 C CNN
 F 2 "" H 7300 4500 60  0000 C CNN
@@
 $EndComp
 $Comp
-L GND #PWR26
+L GND #PWR020
 U 1 1 55D3B956
 P 7700 4500
-F 0 "#PWR26" H 7700 4500 30  0001 C CNN
+F 0 "#PWR020" H 7700 4500 30  0001 C CNN
 F 1 "GND" H 7700 4430 30  0001 C CNN
 F 2 "" H 7700 4500 60  0000 C CNN
@@
 $EndComp
 $Comp
-L GND #PWR27
+L GND #PWR021
 U 1 1 55D3B9B2
 P 8300 4500
-F 0 "#PWR27" H 8300 4500 30  0001 C CNN
+F 0 "#PWR021" H 8300 4500 30  0001 C CNN
 F 1 "GND" H 8300 4430 30  0001 C CNN
 F 2 "" H 8300 4500 60  0000 C CNN
@@
 $EndComp
 $Comp
-L GND #PWR28
+L GND #PWR022
 U 1 1 55D3BA0E
 P 8700 4500
-F 0 "#PWR28" H 8700 4500 30  0001 C CNN
+F 0 "#PWR022" H 8700 4500 30  0001 C CNN
 F 1 "GND" H 8700 4430 30  0001 C CNN
 F 2 "" H 8700 4500 60  0000 C CNN
@@
 $EndComp
 $Comp
-L GND #PWR19
+L GND #PWR023
 U 1 1 55D3BB43
 P 4100 5350
-F 0 "#PWR19" H 4100 5350 30  0001 C CNN
+F 0 "#PWR023" H 4100 5350 30  0001 C CNN
 F 1 "GND" H 4100 5280 30  0001 C CNN
 F 2 "" H 4100 5350 60  0000 C CNN
@@
 $EndComp
 $Comp
-L GND #PWR18
+L GND #PWR024
 U 1 1 55D3BD37
 P 2700 3300
-F 0 "#PWR18" H 2700 3300 30  0001 C CNN
+F 0 "#PWR024" H 2700 3300 30  0001 C CNN
 F 1 "GND" H 2700 3230 30  0001 C CNN
 F 2 "" H 2700 3300 60  0000 C CNN
@@
 $EndComp
 $Comp
-L GND #PWR17
+L GND #PWR025
 U 1 1 55D3BD93
 P 2300 3300
-F 0 "#PWR17" H 2300 3300 30  0001 C CNN
+F 0 "#PWR025" H 2300 3300 30  0001 C CNN
 F 1 "GND" H 2300 3230 30  0001 C CNN
 F 2 "" H 2300 3300 60  0000 C CNN
@@
 $EndComp
 $Comp
-L GND #PWR16
+L GND #PWR026
 U 1 1 55D3BDEF
 P 1600 3250
-F 0 "#PWR16" H 1600 3250 30  0001 C CNN
+F 0 "#PWR026" H 1600 3250 30  0001 C CNN
 F 1 "GND" H 1600 3180 30  0001 C CNN
 F 2 "" H 1600 3250 60  0000 C CNN
@@
 $EndComp
 $Comp
-L GND #PWR22
+L GND #PWR027
 U 1 1 55D3BE67
 P 5450 3250
-F 0 "#PWR22" H 5450 3250 30  0001 C CNN
+F 0 "#PWR027" H 5450 3250 30  0001 C CNN
 F 1 "GND" H 5450 3180 30  0001 C CNN
 F 2 "" H 5450 3250 60  0000 C CNN
@@
 L C-0603 C8
 U 1 1 55D418C9
-P 4350 3100
-F 0 "C8" H 4237 3050 50  0000 R CNN
-F 1 "100n" H 4237 3150 50  0000 R CNN
-F 2 "IPC7351-Nominal:CAPC1608X55" H 4350 3100 50  0001 C CNN
-F 3 "" H 4340 3075 60  0000 C CNN
-F 4 "Value" H 4350 3100 60  0001 C CNN "Manuf"
-F 5 "CAP MLCC 100n ≥X5R 35V 10% [0603]" H 5150 3650 60  0001 C CNN "BOM"
-	1    4350 3100
+P 4450 3100
+F 0 "C8" H 4337 3050 50  0000 R CNN
+F 1 "100n" H 4337 3150 50  0000 R CNN
+F 2 "IPC7351-Nominal:CAPC1608X55" H 4450 3100 50  0001 C CNN
+F 3 "" H 4440 3075 60  0000 C CNN
+F 4 "Value" H 4450 3100 60  0001 C CNN "Manuf"
+F 5 "CAP MLCC 100n ≥X5R 35V 10% [0603]" H 5250 3650 60  0001 C CNN "BOM"
+	1    4450 3100
 	-1   0    0    1
 $EndComp
 Wire Wire Line
-	4350 3000 4350 2900
-Connection ~ 4350 2900
-$Comp
-L GND #PWR20
+	4450 3000 4450 2900
+Connection ~ 4450 2900
+$Comp
+L GND #PWR028
 U 1 1 55D41998
-P 4350 3250
-F 0 "#PWR20" H 4350 3250 30  0001 C CNN
-F 1 "GND" H 4350 3180 30  0001 C CNN
-F 2 "" H 4350 3250 60  0000 C CNN
-F 3 "" H 4350 3250 60  0000 C CNN
-	1    4350 3250
-	1    0    0    -1
-$EndComp
-Wire Wire Line
-	4350 3250 4350 3200
+P 4450 3250
+F 0 "#PWR028" H 4450 3250 30  0001 C CNN
+F 1 "GND" H 4450 3180 30  0001 C CNN
+F 2 "" H 4450 3250 60  0000 C CNN
+F 3 "" H 4450 3250 60  0000 C CNN
+	1    4450 3250
+	1    0    0    -1
+$EndComp
+Wire Wire Line
+	4450 3250 4450 3200
 $Comp
 L TESTPOINT TP?
@@
 Connection ~ 8800 4100
 $Comp
-L PWR #PWR29
+L PWR #PWR029
 U 1 1 55D49638
 P 8900 4050
-F 0 "#PWR29" H 8900 4050 50  0001 C CNN
+F 0 "#PWR029" H 8900 4050 50  0001 C CNN
 F 1 "PWR" H 8900 4050 50  0001 C CNN
 F 2 "" H 8900 4050 60  0000 C CNN
@@
 Connection ~ 9100 4100
 $Comp
-L GND #PWR30
+L GND #PWR030
 U 1 1 55D4D0A0
 P 9100 4500
-F 0 "#PWR30" H 9100 4500 30  0001 C CNN
+F 0 "#PWR030" H 9100 4500 30  0001 C CNN
 F 1 "GND" H 9100 4430 30  0001 C CNN
 F 2 "" H 9100 4500 60  0000 C CNN

Commit message: Finish PCB
Parts:
- removed C10: 220p, IPC7351-Nominal:CAPC1608X55, symbol C-0603
- removed Q3, Q4: 3904, smd-semi:SOT-23, symbol MMBT3904
- removed Q5, Q6: 4403, smd-semi:SOT-23, symbol MMBT4403
- removed R10, R8, R9: 2k, IPC7351-Nominal:RESC1608X50, symbol R-0603
- removed R11, R12: 100, IPC7351-Nominal:RESC1608X50, symbol R-0603
- removed R7: 22k, IPC7351-Nominal:RESC1608X50, symbol R-0603
- added C10: 220p, IPC7351-Nominal:CAPC1005X55, symbol C-0402
- added Q3, Q4: 3904, smd-semi:SC-70, symbol PMSS3904
- added Q5, Q6: 4403, smd-semi:SC-70, symbol PMST4403
- added R10, R8, R9: 2k, IPC7351-Nominal:RESC1005X40, symbol R-0402
- added R11, R12: 100, IPC7351-Nominal:RESC1005X40, symbol R-0402
- added R7: 22k, IPC7351-Nominal:RESC1005X40, symbol R-0402
Connections:
- net GND: now also C10.1, Q6.3, R9.2
- net PREF2: now also R12.2
- net P_OUT: now also R12.1
- net SW: now also Q3.1
- net SWNODE: now also R11.2
- net V+F: now also Q5.2, R10.1, R7.1
- net at Q7.2 (G2), Q7.4 (G1): now also Q4.2, Q5.3, Q6.2
- new net: Q4.3, Q5.1, R10.2
- new net: Q3.3, Q4.1, Q6.1, R7.2
- new net: Q3.2, R8.1
- new net: R8.2, R9.1
- new net: C10.2, R11.1
Other:
- note added: "CRITICAL LAYOUT - These grounds must be connected together with very low impedance."
- note removed: "CRITICAL LAYOUT - These grounds must return with very\nlow inductance to the switching node ground."
