File: Linear.sch (KiCad schematic (older format))
At the start: 61 parts, among them Q10 D45H11, Q11 PMSS3904, Q12 PZT3904, Q8 4403, Q9 2N7002PW, U1 OPA2376AIDGK, U2 LM358DGK, U3 LM393M, U4 LM393M

Commit message: Update schematic to new symbols
Other:
- moved on the sheet: D3, D4
