File: mod12003.kicad_pcb (KiCad board)
At the start: 2 copper layers, 90 x 90 mm, 464 parts, among them J1 IN, J2 OUT, J3 IN, J4 OUT+, J5 OUT-, J6 PDI, J7 BUTTONS, J8 DEVEL, Q1 AO4805, Q10 D45H11, Q11 MMBT3904, Q12 PZT3904, Q2 12A, Q3 3904, Q4 3904, Q5 4403, Q6 4403, Q7 AO4805, Q8 4403, Q9 2N7002PW, U1 OPA2376AID, U10 LM7705, U12 Si8421, U2 LM358M, U3 LM393M, U4 LM393M, U5 ATXMEGA8E5-AU, U6 MCP9701-E/TO, U7 ADR380, U8 AOZ1282, U9 TLV70233DBV

Commit message: Remove OSHW logo
Parts:
- removed SYM1: OSHW-SCHEM-PCB6mm, mech:OSHW-6mm

Commit message: Finish PCB
Parts:
- removed the REF**1111111 at (64.0, 27.5)
- removed the REF**1111111 at (63.0, 27.5)
- removed the REF**1111111 at (62.0, 27.5)
- removed REF**11111111, REF**11111123, REF**11111143, VIA13, VIA14, VIA23 (x2), VIA24 (x2), VIA31: VIA-0.8mm, VIA-0.8mm
- removed the REF**11111131 at (82.5, 53.2)
- removed the REF**1111211 at (40.0, 56.5)
- removed the REF**1111211 at (38.5, 56.5)
- removed the REF**1111211 at (38.5, 55.0)
- removed the REF**1111211 at (43.0, 45.0)
- removed the REF**1111211 at (42.0, 46.0)
- removed the REF**1111211 at (43.2, 49.8)
- removed the REF**1111212 at (32.5, 55.0)
- removed the REF**111123 at (54.5, 55.5)
- removed the VIA11 at (75.5, 32.5)
- removed the VIA12 at (75.5, 34.5)
- removed the VIA21 at (88.5, 32.5)
- removed the VIA21 at (77.5, 32.5)
- removed the VIA22 at (88.5, 34.5)
- removed the VIA22 at (77.5, 34.5)
- removed the VIA5 at (64.0, 18.0)
- removed the VIA5 at (63.0, 18.0)
- removed the VIA5 at (62.0, 18.0)
- added C59: 100n, IPC7351-Nominal:CAPC1005X55, F.Cu at (69.0, 48.5)
- added E6: 120, IPC7351-Nominal:INDC1608X95, F.Cu at (51.5, 40.5)
- added REF**11111131: VIA-0.8mm, VIA-0.8mm, F.Cu at (82.0, 32.5)
- added REF**11111131: VIA-0.8mm, VIA-0.8mm, F.Cu at (82.0, 38.5)
- added REF**11111131: VIA-0.8mm, VIA-0.8mm, F.Cu at (82.0, 57.5)
- added REF**11111131: VIA-0.8mm, VIA-0.8mm, F.Cu at (82.0, 51.5)
- added REF**12132: VIA-0.8mm, VIA-0.8mm, F.Cu at (42.5, 47.0)
- added REF**12132: VIA-0.8mm, VIA-0.8mm, F.Cu at (43.5, 48.0)
- added REF**12132: VIA-0.8mm, VIA-0.8mm, F.Cu at (44.5, 47.0)
- added REF**12132: VIA-0.8mm, VIA-0.8mm, F.Cu at (43.5, 46.0)
- added REF**12132: VIA-0.8mm, VIA-0.8mm, F.Cu at (43.5, 47.0)
- added REF**12144: VIA-0.8mm, VIA-0.8mm, F.Cu at (31.0, 17.0)
- added REF**12144: VIA-0.8mm, VIA-0.8mm, F.Cu at (31.0, 18.0)
- added REF**12144: VIA-0.8mm, VIA-0.8mm, F.Cu at (31.0, 19.0)
- added REF**12144: VIA-0.8mm, VIA-0.8mm, F.Cu at (30.0, 18.5)
- added REF**12144: VIA-0.8mm, VIA-0.8mm, F.Cu at (32.0, 18.5)
- added U11: MAX5215, IPC7351-Nominal:SOP65P490X110-8, F.Cu at (64.5, 48.5)
- added VIA5: VIA-0.8mm, VIA-0.8mm, F.Cu at (58.8, 22.2)
- added VIA5: VIA-0.8mm, VIA-0.8mm, F.Cu at (58.0, 21.8)
- added VIA5: VIA-0.8mm, VIA-0.8mm, F.Cu at (58.8, 21.2)
- C10, C17, C18, C19, C2, C20, C21, C23, C25, C27, C28, C29, C3, C30, C31, C32, C33, C34, C35, C36, C37, C38, C39, C45, C47, C52, C53, C54, C57: footprint IPC7351-Nominal:CAPC1608X55 -> IPC7351-Nominal:CAPC1005X55
- J3: value IN -> 24V
- Q11: value MMBT3904 -> PMSS3904; footprint smd-semi:SOT-23 -> smd-semi:SC-70
- Q3, Q4, Q5, Q6: footprint smd-semi:SOT-23 -> smd-semi:SC-70
- R1, R10, R11, R12, R13, R14, R15, R16, R17, R18, R19, R2, R20, R21, R22, R23, R24, R25, R26, R27, R29, R30, R31, R32, R33, R34, R35, R36, R37, R38, R39, R4, R40, R42, R43, R44, R45, R46, R47, R48, R49, R50, R51, R52, R53, R7, R8, R9: footprint IPC7351-Nominal:RESC1608X50 -> IPC7351-Nominal:RESC1005X40
- R41: value 22k -> 470k; footprint IPC7351-Nominal:RESC1608X50 -> IPC7351-Nominal:RESC1005X40
- U1: value OPA2376AID -> OPA2376AIDGK; footprint IPC7351-Nominal:SOIC127P600X175-8 -> IPC7351-Nominal:SOP65P490X110-8
- U2: value LM358M -> LM358DGK; footprint IPC7351-Nominal:SOIC127P600X175-8 -> IPC7351-Nominal:SOP65P490X110-8
- U5: value ATXMEGA8E5-AU -> ATXMEGA32E5-M4U; footprint IPC7351-Nominal:QFP80P900X900X120-32 -> smd-semi:QFN40P400X400X55-33
- moved J6 27.3 mm to (43.5, 41.5)
- moved R39 23.4 mm to (46.5, 41.5)
- moved U6 22.0 mm to (53.0, 57.0), turned to 0 degrees
- moved R15 10.6 mm to (73.5, 45.8)
- moved R16 10.6 mm to (73.5, 44.2)
- moved TP4 9.30 mm to (31.5, 59.0)
- moved R13 7.54 mm to (73.5, 47.2)
- moved R14 7.54 mm to (73.5, 42.8)
- moved C32 6.58 mm to (48.0, 47.0), turned to 90 degrees
- moved C17 6.52 mm to (71.5, 46.5), turned to 270 degrees
- moved C18 6.52 mm to (71.5, 43.5), turned to 90 degrees
- moved R19 5.52 mm to (69.5, 46.5), turned to 0 degrees
- moved R20 5.52 mm to (69.5, 43.5), turned to 0 degrees
- moved E2 5.50 mm to (49.0, 50.0), turned to 90 degrees
- moved C31 4.95 mm to (39.0, 49.5), turned to 315 degrees
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Connections:
- C10 pad 1: Net-(C10-Pad1) -> GND
- C10 pad 2: GND -> Net-(C10-Pad2)
- C19 pad 1: GND -> Net-(C19-Pad1)
- C19 pad 2: Net-(C19-Pad2) -> GND
- C20 pad 1: GND -> +3.3A
- C20 pad 2: +3.3 -> GND
- C21 pad 1: GND -> V-
- C21 pad 2: V- -> GND
- C23 pad 1: GND -> V-
- C23 pad 2: V- -> GND
- C3 pad 1: /Linear/ISENSE -> /Linear/SCR_FIRE
- C3 pad 2: /Linear/SCR_FIRE -> /Linear/ISENSE
- C31 pad 1: GND -> +3.3
- C31 pad 2: +3.3 -> GND
- C32 pad 1: GND -> +3.3A
- C32 pad 2: +3.3A -> GND
- C33 pad 1: REFGND -> Net-(C33-Pad1)
- C33 pad 2: +3.3A -> REFGND
- C34 pad 1: REFGND -> /Control/VREF
- C34 pad 2: /Control/VREF -> REFGND
- C35 pad 1: GND -> /Control/OVP_THRESH
- C35 pad 2: /Control/OVP_THRESH -> GND
- C36 pad 1: REFGND -> /Control/VSET
- C36 pad 2: /Control/VSET -> REFGND
- C37 pad 1: GND -> /Control/BTN2
- C37 pad 2: Net-(C37-Pad2) -> GND
- C38 pad 1: REFGND -> /Control/ISET
- C38 pad 2: /Control/ISET -> REFGND
- C39 pad 1: GND -> /Control/BTN1
- C39 pad 2: Net-(C39-Pad2) -> GND
- J7 pad 2: Net-(C39-Pad2) -> /Control/BTN1
- J7 pad 3: Net-(C37-Pad2) -> /Control/BTN2
- R11 pad 1: /Preregulator/SWNODE -> Net-(C10-Pad2)
- R11 pad 2: Net-(C10-Pad1) -> /Preregulator/SWNODE
- R17 pad 1: Net-(C19-Pad2) -> Net-(C19-Pad1)
- R24 pad 1: Net-(Q8-Pad1) -> Net-(R24-Pad1)
- R24 pad 2: Net-(R24-Pad2) -> Net-(Q8-Pad1)
- R29 pad 1: V+ -> /Control/~EN
- R29 pad 2: /Control/~EN -> V+
- R30 pad 1: /Linear/P_IN -> Net-(D4-Pad2)
- R30 pad 2: Net-(D4-Pad2) -> /Linear/P_IN
- R37 pad 1: Net-(R36-Pad1) -> GND
- R37 pad 2: GND -> Net-(R36-Pad1)
- R43 pad 2: REFGND -> GND
- R44 pad 1: Net-(R44-Pad1) -> /Control/ISET
- R44 pad 2: /Control/ISET -> Net-(R44-Pad2)
- R45 pad 1: Net-(R45-Pad1) -> /Control/VSET
- R45 pad 2: /Control/VSET -> Net-(R45-Pad2)
- R46 pad 1: Net-(R46-Pad1) -> /Control/LEDCC
- R47 pad 1: Net-(R47-Pad1) -> /Control/LEDCV
- U1 pad 8: +3.3 -> +3.3A
- U4 pad 1: Net-(R24-Pad2) -> Net-(R24-Pad1)
- U4 pad 3: Net-(C19-Pad2) -> Net-(C19-Pad1)
- U5 pad 10: GND -> /Control/~EN
- U5 pad 11: /Control/~EN -> /Control/~VLIM
- U5 pad 12: /Control/~VLIM -> /Control/~ILIM
- U5 pad 13: /Control/~ILIM -> /Control/~SCR_TRIPPED
- U5 pad 14: /Control/~SCR_TRIPPED -> /Control/PREREG_SW
- U5 pad 15: /Control/PREREG_SW -> /Control/OVPTH_PWM
- U5 pad 16: /Control/OVPTH_PWM -> Net-(U5-Pad16)
- U5 pad 19: GND -> Net-(U5-Pad19)
- U5 pad 20: GND -> /Control/BTN1
- U5 pad 21: /Control/TEMP -> /Iso/TO_ISO_OUT
- U5 pad 22: +3.3 -> /Control/RX
- U5 pad 23: +3.3 -> /Control/BTN2
- U5 pad 25: /Iso/TO_ISO_OUT -> /Control/LEDCC
- U5 pad 26: /Control/RX -> /Control/LEDCV
- U5 pad 27: Net-(C37-Pad2) -> /Control/SCL
- U5 pad 28: Net-(C39-Pad2) -> /Control/SDA
- U5 pad 29: Net-(R46-Pad1) -> /Control/TEMP
- U5 pad 3: Net-(R45-Pad1) -> /Control/ISENSE
- U5 pad 30: Net-(R47-Pad1) -> Net-(U5-Pad30)
- U5 pad 31: /Control/ISENSE -> Net-(U5-Pad31)
- U5 pad 4: Net-(R44-Pad1) -> Net-(R44-Pad2)
- U7 pad 1: +3.3A -> Net-(C33-Pad1)
Routing:
- net /Control/BTN1: track 0.00 -> 77.3 mm, vias 0 -> 3
- net /Control/BTN2: track 0.00 -> 76.4 mm
- net Net-(C37-Pad2): track 74.4 -> 0.00 mm
- net Net-(C39-Pad2): track 73.2 -> 0.00 mm
- net /Control/LEDCC: track 0.00 -> 60.6 mm
- net Net-(R46-Pad1): track 57.1 -> 0.00 mm
- net /Control/LEDCV: track 0.00 -> 55.0 mm
- net Net-(R47-Pad1): track 51.9 -> 0.00 mm
- net +3.3: track 182.4 -> 141.0 mm, vias 10 -> 12
- net Net-(R45-Pad1): track 31.9 -> 0.00 mm
- net /Control/PDI_D: track 37.2 -> 9.92 mm, vias 2 -> 0
- net /Linear/P_OUT: track 83.1 -> 58.7 mm
- net /Control/SCL: track 0.00 -> 24.2 mm
- net +3.3A: track 26.0 -> 49.5 mm, vias 2 -> 4
- net /Control/PDI_C: track 31.6 -> 11.0 mm, vias 2 -> 0
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Other:
- net class Default: clearance 0.2 -> 0.195; trace_width 0.3 -> 0.2
- rule trace_clearance: 0.2 -> 0.195
- board text added: "20V 3A SW+LIN"
- board text added: "C D G +"
- board text added: "GEN PURP PSU MODULE"
- board text added: "REV A: 201509"
- board text removed: "--"
- board text removed: "20V 3A PSU MODULE"
- board text removed: "CLK"
- board text removed: "CPOHL1.0 NIHLABS MOD12003 REV A: 201508 ASSY REV:"
- board text removed: "DAT"
- board text removed: "INSUL SCREW ONLY!"
- board text removed: "STAR"
- board text removed: "~RST"

Commit message: Update schematic to new symbols
Parts:
- C58: value 1k/1kV -> 1n/1kV
- DS1: value CC -> CV
- DS2: value CV -> CC
Connections:
- C28 pad 2: Net-(C28-Pad2) -> /Control/FORCE_SAT_L
- D1 pad A: /Linear/ISENSE -> (no net)
- D1 pad K: /Linear/P_OUT -> (no net)
- Q11 pad 3: /Linear/P_IN -> V+
- R25 pad 1: Net-(C28-Pad2) -> /Control/FORCE_SAT_L
- R26 pad 1: Net-(C28-Pad2) -> /Control/FORCE_SAT_L
- R30 pad 2: /Linear/P_IN -> V+
- U2 pad 6: Net-(C28-Pad2) -> /Control/FORCE_SAT_L
- U5 pad 31: Net-(U5-Pad31) -> /Control/FORCE_SAT_L
Routing:
- net /Control/FORCE_SAT_L: track 0.00 -> 8.69 mm
- net Net-(C28-Pad2): track 6.48 -> 0.00 mm
- net V+: track 135.5 -> 139.3 mm
- net /Linear/P_IN: track 78.1 -> 74.4 mm
- net Net-(U5-Pad31): track 2.21 -> 0.00 mm
